File: GraduateProject/CONNECTORS.kicad_sch (KiCad schematic)
At the start: 62 parts, among them J2 Conn_01x05_Pin, J3 Conn_01x05_Pin, J4 Conn_01x04_Pin, J6 Conn_01x04_Pin, Q10 IMX1T110, Q11 IMX1T110, Q12 IMX1T110, Q2 BST50,115, Q3 IMX1T110, Q4 IMX1T110, Q5 IMT2AT108, Q6 IMT2AT108, Q7 IMX1T110, Q8 IMX1T110, Q9 IMX1T110

Commit message: Add files via upload
10/9/25
Parts:
- removed Q5, Q6: IMT2AT108, easyeda2kicad:SOT-457-6_L2.9-W1.7-P0.95-LS2.8-BR, symbol easyeda2kicad:IMT2AT108
- added Q16, Q5: UMT1NTN, easyeda2kicad:SC-70-6_L2.2-W1.3-P0.65-LS2.1-TL, symbol easyeda2kicad:UMT1NTN
- J5: renamed from J6; footprint (none) -> Connector_PinHeader_2.54mm:PinHeader_1x04_P2.54mm_Vertical
- J6: renamed from J4; footprint (none) -> Connector_PinHeader_2.54mm:PinHeader_1x04_P2.54mm_Vertical
- J7: renamed from J3; footprint (none) -> Connector_PinHeader_2.54mm:PinHeader_1x05_P2.54mm_Vertical
- J8: renamed from J2; footprint (none) -> Connector_PinHeader_2.54mm:PinHeader_1x05_P2.54mm_Vertical
- renumbered C14 to C13, C15 to C14, C21 to C15, C181 to C16, C18 to C17, C20 to C18, C1 to C19, C19 to C20, C18 to C21, C17 to C22, C16 to C23, D1 to D7, D2 to D8, Q4 to Q10, Q2 to Q11, Q11 to Q12, Q12 to Q13, Q10 to Q14, Q9 to Q15, Q7 to Q6, Q3 to Q7, Q8 to Q9, R3 to R27, R4 to R28, R2 to R29, R1 to R30, R11 to R31, R9 to R32, R8 to R33, R12 to R34, R13 to R35, R14 to R36, R15 to R37, R10 to R38, R5 to R39, R6 to R40, R7 to R41, R20 to R42, R331 to R43, R32 to R44, R33 to R45, R36 to R46, R49 to R47, R54 to R48, R53 to R49, R52 to R50, R46 to R51, R48 to R52, R51 to R53, R21 to R54, R47 to R55, R50 to R56, R39 to R57, R38 to R58, R37 to R59, TU2 to TU7
Connections:
- net CONN_J2_3: now also Q5.6 (C1)
- net CONN_J2_5: now also Q16.3 (C2)
- net at R27.1: now also Q5.1 (E1)
- net at R31.2: now also Q5.2 (B1), Q5.3 (C2), Q5.5 (B2)
- net at R29.1: now also Q5.4 (E2)
- net at R33.1: now also Q16.2 (B1), Q16.5 (B2), Q16.6 (C1)
- net at R32.2: now also Q16.4 (E2)
- net at R38.2: now also Q16.1 (E1)
Other:
- moved on the sheet: C13, C14, C15, C16, C17, C18, C19, C20, C21, C22, C23, D7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

Commit message: Add files via upload
11/9/25
Parts:
- removed Q11: BST50,115, easyeda2kicad:SOT-89-3_L4.5-W2.5-P1.50-LS4.0-TR, symbol easyeda2kicad:BST50,115
- removed Q16, Q5: UMT1NTN, easyeda2kicad:SC-70-6_L2.2-W1.3-P0.65-LS2.1-TL, symbol easyeda2kicad:UMT1NTN
- added Q3, Q5: DC0150BDJ-7, Package_TO_SOT_SMD:SOT-963, symbol MYLIBS:DC0150BDJ-7
- added Q4: BCX56 AS1-NPN, Package_TO_SOT_SMD:SOT-89-3, symbol Transistor_BJT:BCX56
- D7, D8: value ZMM15_C179550 -> ZMM15_C179550 15V
Connections:
- net CONN_J2_3: now also Q5.1
- net CONN_J2_5: now also Q3.4
- net at C13.1, J7.2 (Pin_2), R36.2: now also Q4.2 (C)
- net at R43.1, R44.1, R46.1: now also Q4.1 (B)
- net at R27.1: now also Q5.6
- net at R33.1: now also Q3.3, Q3.5, Q3.6
- net at R31.2: now also Q5.2, Q5.3, Q5.4
- net at R29.1: now also Q5.5
- net at R38.2: now also Q3.1
- net at R32.2: now also Q3.2
- net at R45.1: now also Q4.3 (E)
Other:
- moved on the sheet: R27, R29, R31, R45

Commit message: Add files via upload
17h37 11/9/2025
Parts:
- removed Q3, Q5: DC0150BDJ-7, Package_TO_SOT_SMD:SOT-963, symbol MYLIBS:DC0150BDJ-7
- removed Q4: BCX56 AS1-NPN, Package_TO_SOT_SMD:SOT-89-3, symbol Transistor_BJT:BCX56
- added Q16, Q17, Q18, Q19, Q2, Q20, Q21, Q22, Q24, Q25, Q27, Q28, Q29, Q30, Q31, Q32, Q33, Q34, Q35: MMBT2222A, Package_TO_SOT_SMD:SOT-23, symbol Transistor_BJT:MMBT2222A
- added Q23, Q26: MMBT3906, Package_TO_SOT_SMD:SOT-23, symbol Transistor_BJT:MMBT3906
- added Q3, Q8: MBT3946DW1T1, Package_TO_SOT_SMD:SOT-363_SC-70-6, symbol Transistor_BJT:MBT3946DW1T1
- Q10, Q12, Q13, Q14, Q15, Q6, Q7, Q9: now not fitted
Connections:
- net CONN_J2_3: now also Q25.2 (E), Q3.1 (E1)
- net CONN_J2_5: now also Q23.2 (E), Q8.4 (E2)
- net GND: now also Q17.1 (B), Q18.1 (B), Q32.1 (B), Q35.1 (B)
- net RA2_PIC1: now also Q16.2 (E), Q31.2 (E)
- net RA2_PIC2: now also Q33.2 (E), Q34.2 (E)
- net RB3_PIC1: now also Q27.1 (B)
- net RB3_PIC2: now also Q21.3 (C)
- net RB4_PIC1: now also Q28.1 (B)
- net RB4_PIC2: now also Q22.3 (C)
- net RB6_PIC1: now also Q31.3 (C)
- net RB6_PIC2: now also Q34.3 (C)
- net RB7_PIC1: now also Q16.3 (C)
- net RB7_PIC2: now also Q33.3 (C)
- net Q7_B1: now reaches J5.2 (Pin_2), Q7.5 (B1), R40.2
- net Q7_B1: now also Q19.1 (B)
- net Q5_2: now reaches R31.2
- net Q5_2: now also Q25.1 (B), Q26.2 (E), Q26.3 (C), Q3.2 (B1), Q3.3 (C2), Q3.4 (E2)
- net Q5_5: now reaches R29.1
- net Q5_5: now also Q26.1 (B), Q3.5 (B2)
- net Q5_6: now reaches R27.1
- net Q5_6: now also Q25.3 (C), Q3.6 (C1)
- net Q6_E1: now reaches J6.1 (Pin_1), Q6.6 (E1)
- net Q6_E1: now also Q27.2 (E)
- net Q9_B2: now reaches J6.2 (Pin_2), Q9.2 (B2), R28.2
- net Q9_B2: now also Q30.1 (B)
- net Q6_E2: now reaches J6.3 (Pin_3), Q6.3 (E2)
- net Q6_E2: now also Q28.2 (E)
- net Q9_B1: now reaches J6.4 (Pin_4), Q9.5 (B1), R35.2
- net Q9_B1: now also Q29.1 (B)
- net Q9_C1: now reaches Q9.1 (C1), Q9.4 (C2), R36.1
- net Q9_C1: now also Q29.3 (C), Q30.3 (C)
- net at C13.1, J7.2 (Pin_2), R36.2: now also Q2.3 (C)
- net Q15_B2: now reaches C23.1, Q15.2 (B2), Q15.6 (E1), R58.1, R59.1
- net Q15_B2: now also Q18.2 (E), Q31.1 (B)
- net Q7_E1: now reaches Q7.6 (E1), R41.2
- net Q7_E1: now also Q19.2 (E)
- net at R43.1, R44.1, R46.1: now also Q2.1 (B)
- net Q3_1: now reaches R38.2
- net Q3_1: now also Q24.2 (E), Q8.1 (E1)
- net Q3_2: now reaches R32.2
- net Q3_2: now also Q24.1 (B), Q8.2 (B1)
- net Q3_3: now reaches R33.1
- net Q3_3: now also Q23.1 (B), Q23.3 (C), Q24.3 (C), Q8.3 (C2), Q8.5 (B2), Q8.6 (C1)
- net Q14_B2: now reaches C22.2, Q14.2 (B2), Q14.6 (E1), R56.1, R57.2
- net Q14_B2: now also Q34.1 (B), Q35.2 (E)
- net Q10_C1: now reaches Q10.1 (C1), Q10.4 (C2), R33.2
- net Q10_C1: now also Q21.1 (B), Q22.1 (B)
- net Q10_E2: now reaches J5.3 (Pin_3), Q10.3 (E2)
- net Q10_E2: now also Q22.2 (E)
- net Q10_E1: now reaches J5.1 (Pin_1), Q10.6 (E1)
- net Q10_E1: now also Q21.2 (E)
- net Q13_B1: now reaches C19.2, Q13.3 (E2), Q13.5 (B1), R47.1, R48.2
- net Q13_B1: now also Q32.2 (E), Q33.1 (B)
- net Q9_E1: now reaches Q9.6 (E1), R34.1
- net Q9_E1: now also Q29.2 (E)
- net at R45.1: now also Q2.2 (E)
- net Q9_E2: now reaches Q9.3 (E2), R37.2
- net Q9_E2: now also Q30.2 (E)
- net Q7_C1: now reaches Q7.1 (C1), Q7.4 (C2), R42.1
- net Q7_C1: now also Q19.3 (C), Q20.3 (C)
- net Q7_B2: now reaches J5.4 (Pin_4), Q7.2 (B2), R39.2
- net Q7_B2: now also Q20.1 (B)
- net Q7_E2: now reaches Q7.3 (E2), R30.2
- net Q7_E2: now also Q20.2 (E)
- net Q6_C1: now reaches Q6.1 (C1), Q6.4 (C2), R31.1
- net Q6_C1: now also Q27.3 (C), Q28.3 (C)
- net Q12_B2: now reaches C15.2, Q12.2 (B2), Q12.6 (E1), R52.1, R55.1
- net Q12_B2: now also Q16.1 (B), Q17.2 (E)
- no-connect marks 7 -> 11
Other:
- moved on the sheet: C13, C14, C15, C16, C17, C18, C19, C20, C21, C22, C23, D7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
