File: GraduateProject/CONNECTORS.kicad_sch (KiCad schematic)
At the start: 82 parts, among them J5 Conn_01x04_Pin, J6 Conn_01x04_Pin, J7 Conn_01x05_Pin, J8 Conn_01x05_Pin, Q10 IMX1T110, Q12 IMX1T110, Q13 IMX1T110, Q14 IMX1T110, Q15 IMX1T110, Q16 MMBT2222A, Q17 MMBT2222A, Q18 MMBT2222A, Q19 MMBT2222A, Q2 MMBT2222A, Q20 MMBT2222A, Q21 MMBT2222A, Q22 MMBT2222A, Q23 MMBT3906, Q24 MMBT2222A, Q25 MMBT2222A, Q26 MMBT3906, Q27 MMBT2222A, Q28 MMBT2222A, Q29 MMBT2222A, Q3 MBT3946DW1T1, Q30 MMBT2222A, Q31 MMBT2222A, Q32 MMBT2222A, Q33 MMBT2222A, Q34 MMBT2222A, Q35 MMBT2222A, Q6 IMX1T110, Q7 IMX1T110, Q8 MBT3946DW1T1, Q9 IMX1T110

Commit message: Add files via upload
13/9/25
Parts:
- R27, R29, R32, R38: value 10R -> 100R
- R40: value 150R -> 330R
Other:
- moved on the sheet: C13, C14, C15, C16, C17, C18, C19, C20, C21, C22, C23, D7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

Commit message: Add files via upload
13h20 22/9/25
Other:
- moved on the sheet: C16, C17, C21, R54, TU7

Commit message: Add files via upload
5/10/25
Parts:
- removed Q2: MMBT2222A, Package_TO_SOT_SMD:SOT-23, symbol Transistor_BJT:MMBT2222A
- added Q37: BCX56, Package_TO_SOT_SMD:SOT-89-3, symbol Transistor_BJT:BCX56
- added Q5: TIP110G, easyeda2kicad:TO-220-3_L10.0-W4.5-P2.54-L, symbol easyeda2kicad:TIP110G
- C13, C14, C15, C16, C17, C18, C20, C21, C22, C23: Buying link (none) -> https://www.thegioiic.com/tu-gom-0805-1-5nf-50v
- C19: Buying link (none) -> https://www.thegioiic.com/tu-gom-0805-68nf-50v
- D7, D8: Buying link (none) -> https://www.thegioiic.com/zmm15-diode-zener-15v-500mw-smd
- Q10, Q12, Q13, Q14, Q15, Q3, Q6, Q7, Q8, Q9: Main Version (none) -> Main
- Q16, Q17, Q18, Q19, Q20, Q21, Q22, Q24, Q25, Q27, Q28, Q29, Q30, Q31, Q32, Q33, Q34, Q35: Buying link (none) -> https://www.thegioiic.com/mmbt2222a-1p-transistor-npn-40v-0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; Split Transistor Version (none) -> Split
- Q23, Q26: Buying link (none) -> https://www.thegioiic.com/mmbt3906-transistor-pnp-40v-0-2a-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; Split Transistor Version (none) -> Split
- R27, R29, R30, R31, R32, R33, R34, R38: Buying link (none) -> https://www.thegioiic.com/dien-tro-100-ohm-0805-1-
- R28, R40: Buying link (none) -> https://www.thegioiic.com/dien-tro-330-ohm-0805-1-
- R35, R39: Buying link (none) -> https://www.thegioiic.com/dien-tro-150-ohm-0805-5-
- R36, R42: Buying link (none) -> https://www.thegioiic.com/dien-tro-470-ohm-0805-1-
- R37, R41, R49, R53: Buying link (none) -> https://www.thegioiic.com/dien-tro-270-ohm-0805-5-
- R43, R45: Buying link (none) -> https://www.thegioiic.com/dien-tro-4-7-ohm-0805-5-
- R44: Buying link (none) -> https://www.thegioiic.com/dien-tro-47-kohm-0805-1-
- R46: Buying link (none) -> https://www.thegioiic.com/dien-tro-1-kohm-0805-1-
- R47, R52, R57, R58: Buying link (none) -> https://www.thegioiic.com/dien-tro-100-kohm-0805-1-
- R48, R55, R56, R59: Buying link (none) -> https://www.thegioiic.com/dien-tro-27-kohm-0805-5-
- R50, R51: Buying link (none) -> https://www.thegioiic.com/dien-tro-10-kohm-0805-1-
- R54: Buying link (none) -> https://www.thegioiic.com/dien-tro-10-ohm-0805-1-
Connections:
- net BCX56_2: now reaches C13.1, J7.2 (Pin_2), R36.2
- net BCX56_2: now also Q37.2 (C), Q5.2 (C)
- net BCX56_1: now reaches R43.1, R44.1, R46.1
- net BCX56_1: now also Q37.1 (B), Q5.1 (B)
- net BCX56_3: now reaches R45.1
- net BCX56_3: now also Q37.3 (E), Q5.3 (E)
- net at J7.1 (Pin_1): now also J7.3 (Pin_3)
- no-connect marks 11 -> 9
Other:
- moved on the sheet: C13, C14, C15, C16, C17, C18, C19, C20, C21, C22, C23, D7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
