File: GraduateProject/GraduateProject.kicad_pcb (KiCad board)
At the start: 2 copper layers, 129 parts, among them IC1 PIC16C620A-04/SS, IC2 PIC16C620A-04/SS, J1 Conn_01x05_Pin, J2 Conn_01x04_Pin, J3 Conn_01x06_Pin, J4 Conn_01x06_Pin, J5 Conn_01x04_Pin, J6 Conn_01x04_Pin, J7 Conn_01x05_Pin, J8 Conn_01x05_Pin, Q1 MMBTRA101SS, Q10 IMX1T110, Q11 BST50,115, Q12 IMX1T110, Q13 IMX1T110, Q14 IMX1T110, Q15 IMX1T110, Q2 MMBTRA101SS, Q3 MMBTRA101SS, Q4 BST50,115, Q5 IMT2AT108, Q6 IMX1T110, Q7 IMX1T110, Q8 IMT2AT108, Q9 IMX1T110, SW1 SS12D10G3, U1 TLP181GB-S, U2 78L05G-AB3-R, U3 78L05G-AB3-R, U4 26V-15V L78L15ABUTR

Commit message: Add files via upload
17h37 11/9/2025
Parts:
- removed D2, D6: BZV55B36, Diode_SMD:D_MiniMELF
- removed J3, J4: Conn_01x06_Pin, Connector_PinHeader_2.54mm:PinHeader_1x06_P2.54mm_Vertical
- removed Q5: IMT2AT108, easyeda2kicad:SOT-457-6_L2.9-W1.7-P0.95-LS2.8-BR
- removed R14, R16: 33k, Resistor_SMD:R_0805_2012Metric
- removed TU5, TU6: 10uF 16V, easyeda2kicad:CAP-SMD_L3.2-W1.6-RD-C7171
- removed U1: TLP181GB-S, easyeda2kicad:SOP-4_L3.7-W4.6-P2.54-LS7.0-TL
- added Q16: MMBT2222A, Package_TO_SOT_SMD:SOT-23, F.Cu at (171.4, 106.9)
- added Q17: MMBT2222A, Package_TO_SOT_SMD:SOT-23, F.Cu at (178.9, 103.8)
- added Q18: MMBT2222A, Package_TO_SOT_SMD:SOT-23, F.Cu at (166.5, 110.0)
- added Q19: MMBT2222A, Package_TO_SOT_SMD:SOT-23, F.Cu at (132.8, 88.5)
- added Q20: MMBT2222A, Package_TO_SOT_SMD:SOT-23, F.Cu at (132.4, 92.3)
- added Q21: MMBT2222A, Package_TO_SOT_SMD:SOT-23, F.Cu at (146.6, 115.7)
- added Q22: MMBT2222A, Package_TO_SOT_SMD:SOT-23, F.Cu at (146.6, 108.2)
- added Q23: MMBT3906, Package_TO_SOT_SMD:SOT-23, F.Cu at (177.6, 115.2)
- added Q24: MMBT2222A, Package_TO_SOT_SMD:SOT-23, F.Cu at (174.3, 112.1)
- added Q25: MMBT2222A, Package_TO_SOT_SMD:SOT-23, F.Cu at (184.3, 121.7)
- added Q26: MMBT3906, Package_TO_SOT_SMD:SOT-23, F.Cu at (184.3, 114.7)
- added Q27: MMBT2222A, Package_TO_SOT_SMD:SOT-23, F.Cu at (148.0, 103.8)
- added Q28: MMBT2222A, Package_TO_SOT_SMD:SOT-23, F.Cu at (155.3, 105.6)
- added Q29: MMBT2222A, Package_TO_SOT_SMD:SOT-23, F.Cu at (171.3, 94.5)
- added Q30: MMBT2222A, Package_TO_SOT_SMD:SOT-23, F.Cu at (163.7, 93.0)
- added Q31: MMBT2222A, Package_TO_SOT_SMD:SOT-23, F.Cu at (164.2, 102.7)
- added Q32: MMBT2222A, Package_TO_SOT_SMD:SOT-23, F.Cu at (141.2, 122.6)
- added Q33: MMBT2222A, Package_TO_SOT_SMD:SOT-23, F.Cu at (138.3, 115.3)
- added Q34: MMBT2222A, Package_TO_SOT_SMD:SOT-23, F.Cu at (154.7, 110.2)
- added Q35: MMBT2222A, Package_TO_SOT_SMD:SOT-23, F.Cu at (161.6, 110.8)
- added Q36: MMBT2222A, Package_TO_SOT_SMD:SOT-23, F.Cu at (141.7, 140.4)
- added U5: B0505S-1W, easyeda2kicad:PWRM-TH_BXXXXS-1W, F.Cu at (149.1, 128.5)
- added U6: EL357N(D)(TA)-G_C42385002, easyeda2kicad:SOP-4_L3.9-W4.4-P2.54-LS7.0-TL, F.Cu at (121.0, 124.5)
- added U7: B0505S-1W, easyeda2kicad:PWRM-TH_BXXXXS-1W, F.Cu at (168.7, 130.8)
- D1, D3, D5: value BZV55B36 -> ZMM36_C8082 35V; footprint Diode_SMD:D_MiniMELF -> easyeda2kicad:LL-34_L3.5-W1.5-RD
- D7, D8: value ZMM15_C179550 -> ZMM15_C179550 15V
- Q1, Q2: value MMBTRA101SS -> MMBT2222A; footprint easyeda2kicad:SOT-23-3_L2.9-W1.3-P1.90-LS2.4-BR -> Package_TO_SOT_SMD:SOT-23
- Q11, Q4: value BST50,115 -> MMBT2222A; footprint easyeda2kicad:SOT-89-3_L4.5-W2.5-P1.50-LS4.0-TR -> Package_TO_SOT_SMD:SOT-23
- Q3: value MMBTRA101SS -> MBT3946DW1T1; footprint easyeda2kicad:SOT-23-3_L2.9-W1.3-P1.90-LS2.4-BR -> Package_TO_SOT_SMD:SOT-363_SC-70-6
- Q8: value IMT2AT108 -> MBT3946DW1T1; footprint easyeda2kicad:SOT-457-6_L2.9-W1.7-P0.95-LS2.8-BR -> Package_TO_SOT_SMD:SOT-363_SC-70-6
- U2: value 78L05G-AB3-R -> L7815; footprint Package_TO_SOT_SMD:SOT-89-3 -> Package_TO_SOT_SMD:TO-263-2
- U3: value 78L05G-AB3-R -> L7805; footprint Package_TO_SOT_SMD:SOT-89-3 -> Package_TO_SOT_SMD:TO-263-2
- U4: value 26V-15V L78L15ABUTR -> L7805; footprint easyeda2kicad:SOT-89-3_L4.5-W2.5-P1.50-LS4.2-TL -> Package_TO_SOT_SMD:TO-263-2
- moved J7 200.2 mm to (192.5, 137.9)
- moved J8 188.3 mm to (192.3, 123.7)
- moved R54 186.5 mm to (188.5, 146.2)
- moved C16 178.4 mm to (188.6, 148.3), turned to 180 degrees
- moved R12 171.5 mm to (180.4, 137.7), turned to 90 degrees
- moved R27 166.8 mm to (187.9, 116.6)
- moved R13 165.7 mm to (175.7, 137.0)
- moved TU7 164.2 mm to (184.5, 146.8), turned to 90 degrees
- moved C20 164.0 mm to (188.8, 128.4), turned to 180 degrees
- moved R29 163.6 mm to (187.9, 118.6)
- moved R49 158.8 mm to (188.5, 124.1)
- moved R53 154.4 mm to (188.8, 130.5), turned to 180 degrees
- moved R15 153.6 mm to (176.3, 124.8), turned to 90 degrees
- moved C18 153.5 mm to (188.8, 126.3)
- moved R46 152.3 mm to (186.8, 108.6)
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Connections:
- net /CONNECTORS/RA2_PIC1 renamed /CONNECTORS/Q12_E2
- net /CONNECTORS/RA2_PIC2 renamed /CONNECTORS/Q13_E1
- net /CONNECTORS/RB3_PIC2 renamed /CONNECTORS/Q10_B1
- net /CONNECTORS/RB4_PIC2 renamed /CONNECTORS/Q10_B2
- net /PICs/ICSPCLK1 renamed /CONNECTORS/Q15_C2
- net /PICs/ICSPCLK2 renamed /CONNECTORS/Q14_C2
- net /PICs/ICSPDAT1 renamed /CONNECTORS/Q12_C2
- net /PICs/ICSPDAT2 renamed /CONNECTORS/Q13_C1
- net /PICs/VPP_!MCLR1 renamed Net-(IC1-~{MCLR}/VPP)
- net /PICs/VPP_!MCLR2 renamed Net-(IC2-~{MCLR}/VPP)
- net Net-(J5-Pin_1) renamed /CONNECTORS/Q10_E1
- net Net-(J5-Pin_2) renamed /CONNECTORS/Q7_B1
- net Net-(J5-Pin_3) renamed /CONNECTORS/Q10_E2
- net Net-(J5-Pin_4) renamed /CONNECTORS/Q7_B2
- net Net-(J6-Pin_1) renamed /CONNECTORS/Q6_E1
- net Net-(J6-Pin_2) renamed /CONNECTORS/Q9_B2
- net Net-(J6-Pin_3) renamed /CONNECTORS/Q6_E2
- net Net-(J6-Pin_4) renamed /CONNECTORS/Q9_B1
- net Net-(Q10-C1) renamed /CONNECTORS/Q10_C1
- net Net-(Q12-B2) renamed /CONNECTORS/Q12_B2
- net Net-(Q13-B1) renamed /CONNECTORS/Q13_B1
- net Net-(Q14-B2) renamed /CONNECTORS/Q14_B2
- net Net-(Q15-B2) renamed /CONNECTORS/Q15_B2
- net Net-(Q6-C1) renamed /CONNECTORS/Q6_C1
- net Net-(Q7-C1) renamed /CONNECTORS/Q7_C1
- net Net-(Q7-E1) renamed /CONNECTORS/Q7_E1
- net Net-(Q7-E2) renamed /CONNECTORS/Q7_E2
- net Net-(Q9-C1) renamed /CONNECTORS/Q9_C1
- net Net-(Q9-E1) renamed /CONNECTORS/Q9_E1
- net Net-(Q9-E2) renamed /CONNECTORS/Q9_E2
- C4 pad 1: Net-(U2-VI) -> Net-(U2-IN)
- C5 pad 1: Net-(U2-VI) -> Net-(U2-IN)
- C7 pad 1: Net-(U2-VI) -> Net-(U2-IN)
- D1 pad 1: Net-(D1-K) -> Net-(D1-C)
- D3 pad 1: +26V -> Net-(D3-C)
- D5 pad 1: /PICs/5V_PIC1 -> +26V
- D5 pad 2: Net-(D5-A) -> GND
- Q1 pad 1: /PICs/RB1_PIC1 -> Net-(Q1-B)
- Q1 pad 3: Net-(D1-K) -> Net-(Q1-C)
- Q11 pad 1: Net-(Q11-E) -> Net-(Q11-B)
- Q11 pad 2: Net-(J7-Pin_2) -> Net-(Q1-C)
- Q11 pad 3: Net-(Q11-B) -> Net-(D1-C)
- Q2 pad 1: Net-(Q2-Pad1) -> Net-(Q2-B)
- Q2 pad 2: Net-(Q2-Pad2) -> Net-(Q2-E)
- Q2 pad 3: Net-(D2-K) -> Net-(J7-Pin_2)
- Q3 pad 1: Net-(Q3-Pad1) -> /CONNECTORS/CONN_J2_3
- Q3 pad 2: GND -> /CONNECTORS/Q5_2
- Q3 pad 3: Net-(Q2-Pad2) -> /CONNECTORS/Q5_2
- Q4 pad 1: Net-(Q4-E) -> Net-(Q4-B)
- Q4 pad 2: /CONNECTORS/CONN_J3_4 -> Net-(Q4-E)
- Q4 pad 3: Net-(Q4-B) -> /CONNECTORS/CONN_J3_4
- Q8 pad 1: /CONNECTORS/CONN_J2_3 -> /CONNECTORS/Q3_1
- Q8 pad 2: Net-(Q8-Pad2) -> /CONNECTORS/Q3_2
- Q8 pad 3: Net-(Q8-Pad2) -> /CONNECTORS/Q3_3
- Q8 pad 4: Net-(Q8-Pad2) -> /CONNECTORS/CONN_J2_5
- Q8 pad 5: Net-(Q8-Pad5) -> /CONNECTORS/Q3_3
- Q8 pad 6: Net-(Q8-Pad6) -> /CONNECTORS/Q3_3
- R13 pad 1: Net-(D5-A) -> Net-(U7-Vo)
- R2 pad 2: Net-(Q2-Pad1) -> Net-(Q11-B)
- R27 pad 1: Net-(Q8-Pad6) -> /CONNECTORS/Q5_6
- R29 pad 1: Net-(Q8-Pad5) -> /CONNECTORS/Q5_5
- R3 pad 2: Net-(Q2-Pad1) -> Net-(Q11-B)
- R31 pad 2: Net-(Q8-Pad2) -> /CONNECTORS/Q5_2
- R32 pad 2: Net-(Q5-Pad5) -> /CONNECTORS/Q3_2
- R33 pad 1: Net-(Q5-Pad1) -> /CONNECTORS/Q3_3
- R38 pad 2: Net-(Q5-Pad6) -> /CONNECTORS/Q3_1
- R4 pad 2: Net-(Q3-Pad1) -> Net-(Q1-B)
- R43 pad 1: Net-(Q11-B) -> Net-(Q2-B)
- R44 pad 1: Net-(Q11-B) -> Net-(Q2-B)
- R45 pad 1: Net-(Q11-E) -> Net-(Q2-E)
- R46 pad 1: Net-(Q11-B) -> Net-(Q2-B)
- R5 pad 2: Net-(Q3-Pad1) -> Net-(Q1-B)
- R8 pad 1: Net-(U2-VI) -> Net-(U2-IN)
- R9 pad 1: Net-(U4-VOUT) -> Net-(U2-OUT)
- REL1 pad A1: Net-(D1-K) -> Net-(D3-C)
- REL2 pad A1: Net-(D2-K) -> Net-(D1-C)
- TU4 pad 1: Net-(U4-VOUT) -> Net-(U2-OUT)
- U2 pad 1: Net-(U2-VI) -> Net-(U2-IN)
- U2 pad 3: /PICs/5V_PIC1 -> Net-(U2-OUT)
- U3 pad 1: Net-(U2-VI) -> Net-(U2-IN)
- U3 pad 3: /PICs/5V_PIC2 -> /PICs/5V_PIC1
- U4 pad 1: Net-(U4-VOUT) -> Net-(U2-IN)
- U4 pad 3: Net-(U2-VI) -> /PICs/5V_PIC2
Routing:
- net /CONNECTORS/Q3_2: track 0.00 -> 2.93 mm
Other:
- board outline added: 90 x 70 mm
- board text added: "10mm"
- board text added: "20mm"
- board text added: "21mm"
- board text added: "2mm"
- board text added: "40mm"
- board text added: "45mm"
- board text added: "48.5mm"
- board text added: "51mm"
- board text added: "70mm"
- board text added: "80mm"
- board text added: "90mm"
- board text added: "9mm"
- board text added: "Phi 2mm"
- board text added: "Phi 3mm"
