File: GraduateProject/GraduateProject.kicad_sch (KiCad schematic)
At the start: 110 parts, among them IC1 PIC16C620A-04/SS, IC2 PIC16C620A-04/SS, IC3 SPX5205M5-L-5-0/TR, IC4 SPX5205M5-L-5-0/TR, J1 Conn_01x05_Pin, J2 Conn_01x05_Pin, Q1 BST50,115, Q1 IMT2AT108, Q10 IMX1T110, Q11 IMX1T110, Q12 IMX1T110, Q13 BC846 1B, Q14 BC846 1B, Q15 BC846 1B, Q2 BST50,115, Q3 IMX1T110, Q4 IMX1T110, Q5 IMT2AT108, Q7 IMX1T110, Q8 IMX1T110, Q9 IMX1T110, SW1 SS12D10G3, U1 26V-15V L78L15ABUTR, U2 78L05G-AB3-R, U3 78L05G-AB3-R, U4 TLP181GB-S

Commit message: Add files via upload
21/8/25
Parts:
- removed Q13, Q14, Q15: BC846 1B, easyeda2kicad:SOT-23-3_L2.9-W1.6-P1.90-LS2.8-BR, symbol easyeda2kicad:BC8461B
- added J3: Conn_01x05_Pin, symbol Connector:Conn_01x05_Pin
- added J4, J5, J6: Conn_01x04_Pin, symbol Connector:Conn_01x04_Pin
- added Q13, Q14, Q15: MMBTRA101SS, easyeda2kicad:SOT-23-3_L2.9-W1.3-P1.90-LS2.4-BR, symbol easyeda2kicad:MMBTRA101SS
- added R20: 470R, Resistor_SMD:R_0805_2012Metric, symbol Device:R
- added R21: 10R, Resistor_SMD:R_0805_2012Metric, symbol Device:R
- added R331: 4.7R, Resistor_SMD:R_0805_2012Metric, symbol Device:R
- added TP1, TP10, TP11, TP12, TP13, TP2, TP3, TP4, TP5, TP8, TP9: TestPoint, symbol Connector:TestPoint
- added TP14, TP15, TP16, TP17, TP18, TP19, TP20, TP21: ?, symbol Connector:TestPoint
- added TP22, TP23, TP6, TP7: GND?, symbol Connector:TestPoint
- added TU2: 3.3uF 35V, easyeda2kicad:CAP-SMD_L3.5-W2.8-R-RD, symbol easyeda2kicad:TAJB335K035RNJ
- renumbered Q1 to Q6
Connections:
- net GND: now also C14.2, C15.2, TP1.1, TP13.1, TP16.1, TP3.1
- net at R6.1: now also C2.2, C9.2, D4.2 (A), IC1.9 (RB2), R1.1, R26.2, R27.2, R28.2, R32.2, R33.2, R5.1, R7.1, TU1.1, J5.2 (Pin_2), R331.2, TP20.1, TP21.1, TP22.1, TP23.1, TP7.1
- net at R6.2: now also Q3.5 (B1), J6.2 (Pin_2)
- net at C1.1, C20.2, J2.2 (Pin_2)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: now also C21.1
- net at C19.1, J2.3 (Pin_3): now also D2.2, Q6.4, TP2.1, TP4.1
- net at C17.1, C18.1, J2.4 (Pin_4)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: now also C16.2
- net at J2.5 (Pin_5): now also C15.1, D1.2, Q5.6, TP15.1
- net at C17.2, Q10.2 (B2), Q10.6 (E1)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: no longer R38.1
- net at R38.2: now also IC2.3 (RA4/T0CKI), Q9.4 (C2), TP12.1
- net at R7.2: now also Q3.6 (E1)
- net at R23.1: now also IC1.1 (RA2/AN2/VREF)
- net at R23.2: now also IC1.2 (RA3/AN3), R24.2, R31.2
- net at R28.1: now also Q1.1 (E), TP19.1
- net at D4.1 (K): now also D3.1 (C), TP6.1
- net at Q4.1 (C1): now also R8.2
- net at Q4.2 (B2): now also IC1.10 (RB3), TP8.1
- net at Q4.3 (E2): now also J6.3 (Pin_3)
- net at Q4.6 (E1): now also J6.1 (Pin_1)
- net at C9.1: now also R25.2
- net at Q12.1 (C1), R49.2: now also IC1.7 (RB0/INT); no longer IC1.14 (RB7)
- net at C2.1: now also D3.2 (A), J5.1 (Pin_1)
- net at Q9.2 (B2): now also C16.1, Q9.6 (E1), R37.1, R38.1
- net at Q9.3 (E2): now also TP10.1
- net at Q9.5 (B1): now also Q11.5 (B1), R37.2, R46.1, R47.2, TP11.1
- net at R32.1: now also Q2.3 (B), R36.1, R331.1
- net at Q3.2 (B2): now also R5.2, J6.4 (Pin_4)
- net at Q3.3 (E2): now also R1.2
- net at R3.2: now also D1.1, D2.1, R10.1, R2.2, R9.1
- net at Q6.1: now also R11.2
- net at Q6.5: now also Q6.6
- net at Q10.4 (C2), R39.1: now also IC1.8 (RB1), TP14.1; no longer IC1.13 (RB6)
- net at Q5.1: now also Q5.5
- net at Q5.2: now also R9.2
- net at Q5.3: now also R10.2
- net at Q5.4: now also R8.1
- net at C12.1: now also IC1.15 (VDD)
- net at C12.2: now also C10.2, C11.1
- net at C10.1: now also IC2.8 (RB1), R42.2
- net at R11.1: now also Q7.1 (C1), Q7.4 (C2)
- net at IC2.1 (RA2/AN2/VREF): now also Q7.2 (B2)
- net at IC2.15 (VDD): now also IC2.16 (VDD)
- net at IC2.2 (RA3/AN3): now also R36.2
- net at IC2.20 (RA1/AN1): now also Q7.5 (B1)
- net at IC2.4 (~{MCLR}/VPP): now also Q11.4 (C2), R48.2, TP9.1
- net at IC2.5 (VSS): now also C11.2, IC2.6 (VSS), R42.1
- net at R26.1: now also R27.1
- net at IC1.4 (~{MCLR}/VPP): now also R24.1, R25.1, TU3.1
- net at IC1.5 (VSS): now also IC1.6 (VSS)
- net at Q2.1 (E): now also R33.1, TP18.1
- net at Q2.2 (C): now also C14.1, J3.2 (Pin_2), TP17.1
- net at R47.1: now also C21.2, Q11.2 (B2), Q11.6 (E1), R48.1
- net at R46.2: now also Q11.3 (E2), TP5.1
- net at Q7.3 (E2): now also J4.2 (Pin_2)
- net at Q7.6 (E1): now also J4.1 (Pin_1)
- no-connect marks 2 -> 3
Other:
- moved on the sheet: C12, C14, C15, C18, IC2, Q1, Q10, Q2, Q3, Q6, Q7, Q8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

Commit message: 2/9/25
Parts:
- removed IC3, IC4: SPX5205M5-L-5-0/TR, easyeda2kicad:SOT-23-5_L3.0-W1.7-P0.95-LS2.8-TL, symbol easyeda2kicad:SPX5205M5-L-5-0_TR
- removed TP1, TP10, TP11, TP12, TP13, TP2, TP3, TP4, TP5, TP8, TP9: TestPoint, symbol Connector:TestPoint
- removed TP14, TP15, TP16, TP17, TP18, TP19, TP20, TP21: ?, symbol Connector:TestPoint
- removed TP22, TP23, TP6, TP7: GND?, symbol Connector:TestPoint
- added C181: 50V 1.5nF, Capacitor_SMD:C_0805_2012Metric, symbol Device:C
- added D7, D8: BZV55B36, Diode_SMD:D_MiniMELF, symbol Diode:BZV55B36
- added R19, R22, R57, R58: 33k, Resistor_SMD:R_0805_2012Metric, symbol Device:R
- added R55: 1k, Resistor_SMD:R_0805_2012Metric, symbol Device:R
- added R56: 100R, Resistor_SMD:R_0805_2012Metric, symbol Device:R
- added TU6, TU7: 10uF 16V, easyeda2kicad:CAP-SMD_L3.2-W1.6-RD-C7171, symbol easyeda2kicad:TAJA106K016RNJ
Connections:
- net GND: now also C10.2, C11.1, C12.2, C18.1, C2.2, C4.2, C5.2, C6.2, C7.2, C8.2, C9.2, D4.2 (A), D5.2 (A), D6.2 (A), IC1.5 (VSS), IC1.6 (VSS), IC2.5 (VSS), IC2.6 (VSS), J5.2 (Pin_2), Q11.5 (B1), Q13.2, Q15.2, Q9.5 (B1), R1.1, R12.2, R13.1, R15.1, R27.2, R28.2, R32.2, R33.2, R331.2, R34.1, R37.2, R4.1, R40.1, R43.2, R46.1, R47.2, R5.1, R6.1, R7.1, REL1.A2, REL2.A2, SW1.1, TU1.1, TU2.2, TU3.2, TU4.2, TU5.2, U1.2 (GND), U2.2 (GND), U3.2 (GND), U4.4 (EMI), C181.2, R19.2, R22.2, TU6.2, TU7.2
- net at R40.2: now also Q14.1, R41.2
- net at R34.2: now also Q13.1, R35.2
- net CONN_J2_3: now reaches C19.1, D2.2, J2.3 (Pin_3)
- net CONN_J2_3: now also Q6.1; no longer Q6.4
- net CONN_J2_4: now reaches C16.2, C17.1, C18.1, J2.4 (Pin_4), R51.1
- net CONN_J2_5: now reaches C15.1, J2.5 (Pin_5)
- net CONN_J2_5: now also D1.1, Q5.3; no longer D1.2, Q5.6
- net at REL1.4: now also J1.2 (Pin_2)
- net at REL1.5: now also J1.3 (Pin_3)
- net at REL1.A1: now also D5.1 (K), Q14.3
- net at U1.1 (VOUT): now also TU3.1, R55.1
- net at U1.3 (VIN): now also C5.1, C6.1, C7.1, R18.1, U2.1 (VI), U3.1 (VI)
- net at J4.2 (Pin_2): now also Q8.2 (B2), R4.2; no longer Q7.3 (E2)
- net at J4.3 (Pin_3): now also Q7.3 (E2)
- net at J4.4 (Pin_4): now also Q8.5 (B1), R13.2
- net at R14.1: now also Q8.1 (C1), Q8.4 (C2)
- net at R14.2: now also C14.1, J3.2 (Pin_2), Q2.2 (C)
- net at R17.1: now also C3.2, R16.2, U4.1 (AN)
- net at R17.2: now also C1.2, C3.1, J5.4 (Pin_4), U4.3 (CAT)
- net RB6_PIC1: now reaches Q9.4 (C2), R38.2
- net RB6_PIC1: now also IC2.13 (RB6); no longer IC2.3 (RA4/T0CKI)
- net at Q13.3: now also Q14.2
- net RA1_AN1: now reaches R23.1
- net RA1_AN1: now also IC1.20 (RA1/AN1), IC2.20 (RA1/AN1), R19.1; no longer IC1.1 (RA2/AN2/VREF)
- net RA0_AN0: now reaches R23.2, R24.2, R31.2
- net RA0_AN0: now also IC1.19 (RA0/AN0), IC2.19 (RA0/AN0); no longer IC1.2 (RA3/AN3)
- net RA4_T0CKI: now reaches C4.1
- net RA4_T0CKI: now also IC1.3 (RA4/T0CKI), IC2.3 (RA4/T0CKI), R30.2, U4.6 (COL)
- net at C17.2, Q10.2 (B2), Q10.6 (E1)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: now also R50.1
- net +26V: now reaches D3.1 (C), D4.1 (K)
- net +26V: now also R18.2, R21.1, TU1.2
- net at Q4.1 (C1), R8.2: now also Q4.4 (C2)
- net RB3: now reaches IC1.10 (RB3)
- net RB3: now also Q4.5 (B1); no longer Q4.2 (B2)
- net at C9.1, R25.2: now also IC1.18 (OSC1/CLKIN)
- net RB7_PIC2: now reaches Q12.1 (C1), R49.2
- net RB7_PIC2: now also IC1.14 (RB7); no longer IC1.7 (RB0/INT)
- net at R12.1: now also Q8.6 (E1)
- net RB1: now reaches Q15.1
- net RB1: now also R43.1, R45.1
- net at Q15.3: now also D6.1 (K), REL2.A1
- net RA2_PIC1: now reaches Q9.3 (E2)
- net RA2_PIC1: now also IC2.1 (RA2/AN2/VREF), Q11.3 (E2), R46.2
- net at R29.1: now also D7.2 (A), R57.2, TU6.1
- net at R29.2: now also IC1.4 (~{MCLR}/VPP)
- net 5V_PIC2: now reaches U2.3 (VO)
- net 5V_PIC2: now also C12.1, IC1.15 (VDD), IC1.16 (VDD), R24.1, R25.1, R30.1, TU4.1, D7.1 (K), R57.1
- net at SW1.2: now also IC1.9 (RB2), IC2.2 (RA3/AN3)
- net 5V_PIC1: now reaches SW1.3
- net 5V_PIC1: now also C11.2, C8.1, IC2.15 (VDD), IC2.16 (VDD), R42.1, TU5.1, U3.3 (VO), D8.1 (K), R58.1
- net at J1.4 (Pin_4): now also REL2.4
- net at J1.5 (Pin_5): now also REL2.5
- net RA2_PIC2: now reaches Q10.3 (E2), Q12.6 (E1), R52.2
- net RA2_PIC2: now also IC1.1 (RA2/AN2/VREF)
- net at Q8.3 (E2): now also R15.2
- net at R45.2: now also IC2.8 (RB1)
- net at Q3.1 (C1): now also Q3.4 (C2), R20.1
- net CONN_J3_4: now reaches Q1.2 (C)
- net CONN_J3_4: now also C18.2, J3.4 (Pin_4), R20.2
- net at Q1.3 (B): now also R26.1, R27.1
- net at R3.1: now also Q6.6
- net 14.5V: now reaches D2.1, R10.1, R2.2, R3.2, R9.1
- net 14.5V: now also D1.2, R22.1, R56.1; no longer D1.1
- net at R11.2: now also Q6.2, Q6.3, Q6.4; no longer Q6.1
- net at Q6.5: now also R2.1; no longer Q6.6
- net RB6_PIC2: now reaches Q10.4 (C2), R39.1
- net RB6_PIC2: now also IC1.13 (RB6); no longer IC1.8 (RB1)
- net at Q5.1: now also Q5.2, Q5.4, R8.1; no longer Q5.5
- net at R9.2: now also Q5.5; no longer Q5.2
- net at R10.2: now also Q5.6; no longer Q5.3
- net at C10.1, R42.2: now also IC2.18 (OSC1/CLKIN); no longer IC2.8 (RB1)
- net RB7_PIC1: now reaches Q11.4 (C2), R48.2
- net RB7_PIC1: now also IC2.14 (RB7); no longer IC2.4 (~{MCLR}/VPP)
- net RB4_PIC1: now reaches Q7.2 (B2)
- net RB4_PIC1: now also IC2.11 (RB4); no longer IC2.1 (RA2/AN2/VREF)
- net RB3_PIC1: now reaches IC2.10 (RB3)
- net RB3_PIC1: now also Q7.5 (B1)
- net RB5_PIC1: now reaches IC2.12 (RB5)
- net RB5_PIC1: now also R36.2
- net RBO/INT: now reaches IC2.7 (RB0/INT)
- net RBO/INT: now also IC1.7 (RB0/INT)
- net RB2_PIC1: now reaches IC2.9 (RB2)
- net RB2_PIC1: now also R35.1
- net CONN_J3_5: now reaches J3.5 (Pin_5)
- net CONN_J3_5: now also R21.2, TU2.1, C181.1
- net RB4_PIC2: now reaches IC1.11 (RB4)
- net RB4_PIC2: now also Q4.2 (B2)
- net at IC1.12 (RB5): now also R26.2
- net at R16.1: now also C1.1, J5.3 (Pin_3)
- net RB1_PIC2: now reaches R41.1
- net RB1_PIC2: now also IC1.8 (RB1)
- net at R44.1: now also D8.2 (A), R58.2, TU7.1
- net at R44.2: now also IC2.4 (~{MCLR}/VPP)
- net at R31.1: now also IC1.2 (RA3/AN3)
- new net: R55.2, R56.2
- no-connect marks 3 -> 12
Other:
- note added: "CONNECTORS"
- note added: "PICs"
- note added: "POWER"
- note added: "RELAYS"
- moved on the sheet: C1, C10, C11, C12, C14, C15, C16, C17, C18, C19, C2, C20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

Commit message: 3/9/25
Parts:
- removed C1: 50V 68nF, Capacitor_SMD:C_0805_2012Metric, symbol Device:C
- removed C1: 50V 68nF ceramic, Capacitor_SMD:C_0805_2012Metric, symbol Device:C
- removed C10, C9: 50V 68pF, Capacitor_SMD:C_0805_2012Metric, symbol Device:C
- removed C11, C12, C4: 50V 10nF, Capacitor_SMD:C_0805_2012Metric, symbol Device:C
- removed C14, C15, C16, C17, C18 (x2), C181, C19, C20, C21, C3, C5, C6, C7, C8: 50V 1.5nF, Capacitor_SMD:C_0805_2012Metric, symbol Device:C
- removed C2: 50V 10nF ceramic, Capacitor_SMD:C_1206_3216Metric, symbol Device:C
- removed D1, D2: ZMM15_C179550, easyeda2kicad:SOD-80_L3.5-W1.5-RD, symbol easyeda2kicad:ZMM15_C179550
- removed D3: FM4007, easyeda2kicad:SOD-123FL_L2.7-W1.8-LS3.8-RD, symbol easyeda2kicad:FM4007
- removed D4, D5, D6, D7, D8: BZV55B36, Diode_SMD:D_MiniMELF, symbol Diode:BZV55B36
- removed IC1, IC2: PIC16C620A-04/SS, easyeda2kicad:SSOP-20_L7.2-W5.3-P0.65-LS7.8-BL, symbol easyeda2kicad:PIC16C620A-04_SS
- removed J1, J2, J3: Conn_01x05_Pin, symbol Connector:Conn_01x05_Pin
- removed J4, J5, J6: Conn_01x04_Pin, symbol Connector:Conn_01x04_Pin
- removed Q1, Q2: BST50,115, easyeda2kicad:SOT-89-3_L4.5-W2.5-P1.50-LS4.0-TR, symbol easyeda2kicad:BST50,115
- removed Q10, Q11, Q12, Q3, Q4, Q7, Q8, Q9: IMX1T110, easyeda2kicad:SOT-457_L2.9-W1.6-P0.95-LS2.80-BR, symbol easyeda2kicad:IMX1T110
- removed Q13, Q14, Q15: MMBTRA101SS, easyeda2kicad:SOT-23-3_L2.9-W1.3-P1.90-LS2.4-BR, symbol easyeda2kicad:MMBTRA101SS
- removed Q5, Q6: IMT2AT108, easyeda2kicad:SOT-457-6_L2.9-W1.7-P0.95-LS2.8-BR, symbol easyeda2kicad:IMT2AT108
- removed R1, R11, R12, R56, R8: 100R, Resistor_SMD:R_0805_2012Metric, symbol Device:R
- removed R10, R18, R2, R21, R3, R9: 10R, Resistor_SMD:R_0805_2012Metric, symbol Device:R
- removed R13, R5, R6: 150R, Resistor_SMD:R_0805_2012Metric, symbol Device:R
- removed R14, R20: 470R, Resistor_SMD:R_0805_2012Metric, symbol Device:R
- removed R15, R51, R53, R7: 270R, Resistor_SMD:R_0805_2012Metric, symbol Device:R
- removed R16, R25, R42: 3.3k, Resistor_SMD:R_0805_2012Metric, symbol Device:R
- removed R17, R19, R22, R57, R58: 33k, Resistor_SMD:R_0805_2012Metric, symbol Device:R
- removed R23, R27, R31, R32: 47k, Resistor_SMD:R_0805_2012Metric, symbol Device:R
- removed R24, R30, R46, R52: 10k, Resistor_SMD:R_0805_2012Metric, symbol Device:R
- removed R26, R29, R35, R36, R41, R43, R44, R45, R55: 1k, Resistor_SMD:R_0805_2012Metric, symbol Device:R
- removed R28, R33, R331: 4.7R, Resistor_SMD:R_0805_2012Metric, symbol Device:R
- removed R34, R40: 4.7k, Resistor_SMD:R_0805_2012Metric, symbol Device:R
- removed R37, R47, R50, R54: 27k, Resistor_SMD:R_0805_2012Metric, symbol Device:R
- removed R38, R39, R48, R49: 100k, Resistor_SMD:R_0805_2012Metric, symbol Device:R
- removed R4: 330R, Resistor_SMD:R_0805_2012Metric, symbol Device:R
- removed REL1, REL2: V23057-B0006-A101, easyeda2kicad:RELAY-TH_TE_V23057BXXX, symbol easyeda2kicad:V23057-B0006-A101
- removed SW1: SS12D10G3, easyeda2kicad:SW-TH_3P-P4.8-L12.7-W6.7_SS12D10G3, symbol easyeda2kicad:SS12D10G3
- removed TU1, TU2: 3.3uF 35V, easyeda2kicad:CAP-SMD_L3.5-W2.8-R-RD, symbol easyeda2kicad:TAJB335K035RNJ
- removed TU3: 2.2uF 35V, easyeda2kicad:CAP-SMD_L3.5-W2.8-R-RD, symbol easyeda2kicad:TAJB225K035RNJ
- removed TU4, TU5, TU6, TU7: 10uF 16V, easyeda2kicad:CAP-SMD_L3.2-W1.6-RD-C7171, symbol easyeda2kicad:TAJA106K016RNJ
- removed U1: 26V-15V L78L15ABUTR, easyeda2kicad:SOT-89-3_L4.5-W2.5-P1.50-LS4.2-TL, symbol easyeda2kicad:L78L15ABUTR
- removed U2, U3: 78L05G-AB3-R, Package_TO_SOT_SMD:SOT-89-3, symbol Regulator_Linear:KA78M05_TO252
- removed U4: TLP181GB-S, easyeda2kicad:SOP-4_L3.7-W4.6-P2.54-LS7.0-TL, symbol easyeda2kicad:TLP181GB-S
Connections:
- no-connect marks 12 -> 0
Other:
- added sheet CONNECTORS (CONNECTORS.kicad_sch)
- added sheet PICs (PICs.kicad_sch)
- added sheet POWER (POWER.kicad_sch)
- added sheet Relays (Relays.kicad_sch)
- note removed: "CONNECTORS"
- note removed: "PICs"
- note removed: "POWER"
- note removed: "RELAYS"

Commit message: Add files via upload
17h37 11/9/2025
Changed lines of the file:
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@@
 	(sheet
 		(at 61.468 100.584)
-		(size 17.272 23.622)
+		(size 17.272 18.796)
 		(exclude_from_sim no)
 		(in_bom yes)
@@
 		)
 		(property "Sheetfile" "Relays.kicad_sch"
-			(at 61.468 124.7906 0)
+			(at 61.468 119.9646 0)
 			(effects
 				(font
