File: GraduateProject/PICs.kicad_sch (KiCad schematic)
At the start: 24 parts, among them IC1 PIC16C620A-04/SS, IC2 PIC16C620A-04/SS, Q4 MMBT2222A, SW1 SS12D10G3, U5 B0505S-1W, U7 B0505S-1W

Commit message: Add files via upload
5/10/25
Parts:
- removed Q4: MMBT2222A, Package_TO_SOT_SMD:SOT-23, symbol Transistor_BJT:MMBT2222A
- added Q2: TIP110G, easyeda2kicad:TO-220-3_L10.0-W4.5-P2.54-L, symbol easyeda2kicad:TIP110G
- added Q38: BCX56, Package_TO_SOT_SMD:SOT-89-3, symbol Transistor_BJT:BCX56
- C10, C11: Buying link (none) -> https://www.thegioiic.com/tu-gom-0805-10nf-50v
- C12, C9: Buying link (none) -> https://www.thegioiic.com/tu-gom-0805-68pf-50v
- C8: Buying link (none) -> https://www.thegioiic.com/tu-gom-0805-1-5nf-50v
- R12, R13, R17, R24: Buying link (none) -> https://www.thegioiic.com/dien-tro-1-kohm-0805-1-
- R15, R23: Buying link (none) -> https://www.thegioiic.com/dien-tro-3-3-kohm-0805-1-
- R18, R20, R25: Buying link (none) -> https://www.thegioiic.com/dien-tro-47-kohm-0805-1-
- R19, R22: Buying link (none) -> https://www.thegioiic.com/dien-tro-10-kohm-0805-1-
- R21: Buying link (none) -> https://www.thegioiic.com/dien-tro-33-kohm-0805-1-
- R26: Buying link (none) -> https://www.thegioiic.com/dien-tro-4-7-ohm-0805-5-
- SW1: Buying link (none) -> https://www.thegioiic.com/ss12d00g4-cong-tac-truot-3-chan-x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
- U5, U7: Buying link (none) -> https://www.thegioiic.com/b0505s-1wr3-chuyen-doi-dc-dc-vao-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
Connections:
- net CONN_J3_4: now also Q2.2 (C), Q38.2 (C)
- net BCX56_38_3: now reaches R26.1
- net BCX56_38_3: now also Q2.3 (E), Q38.3 (E)
- net BCX56_38_1: now reaches R24.1, R25.1
- net BCX56_38_1: now also Q2.1 (B), Q38.1 (B)
Other:
- moved on the sheet: C10, C11, C12, C8, C9, IC1, IC2, R12, R13, R15, R17, R18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
