File: GraduateProject/POWER.kicad_sch (KiCad schematic)
At the start: 24 parts, among them J5 Conn_01x04_Pin, U1 26V-15V L78L15ABUTR, U2 78L05G-AB3-R, U3 78L05G-AB3-R, U4 TLP181GB-S

Commit message: Add files via upload
10/9/25
Parts:
- J2: renamed from J5; footprint (none) -> Connector_PinHeader_2.54mm:PinHeader_1x04_P2.54mm_Vertical
- renumbered C4 to C1, C3 to C2, C2 to C3, C7 to C4, C6 to C5, C2 to C6, C5 to C7, D4 to D3, D3 to D4, R56 to R10, R22 to R11, R17 to R6, R16 to R7, R18 to R8, R55 to R9, TU5 to TU1, TU4 to TU2, TU1 to TU3, TU3 to TU4, U4 to U1, U3 to U2, U2 to U3, U1 to U4

Commit message: Add files via upload
11/9/25
Parts:
- removed D3: BZV55B36, Diode_SMD:D_MiniMELF, symbol Diode:BZV55B36
- added D5: ZMM33_C8082 35V, easyeda2kicad:LL-34_L3.5-W1.5-RD, symbol easyeda2kicad:ZMM33_C8082
Connections:
- net +26V: now also D5.1 (C)
- net GND: now also D5.2 (A)
Changed lines of the file:
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@@
 	(wire
 		(pts
-			(xy 125.73 66.04) (xy 132.08 66.04)
+			(xy 123.19 66.04) (xy 129.54 66.04)
 		)
 		(stroke
@@
 	(wire
 		(pts
-			(xy 125.73 69.85) (xy 125.73 66.04)
+			(xy 123.19 69.85) (xy 123.19 66.04)
 		)
 		(stroke
@@
 	)
 	(symbol
+		(lib_id "easyeda2kicad:ZMM33_C8082")
+		(at 134.62 66.04 180)
+		(unit 1)
+		(exclude_from_sim no)
+		(in_bom yes)
+		(on_board yes)
+		(dnp no)
+		(fields_autoplaced yes)
+		(property "Reference" "D5"
+			(at 135.255 58.42 0)
+			(effects
+				(font
+					(size 1.27 1.27)
+				)
+			)
+		)
+		(property "Value" "ZMM33_C8082 35V"
+			(at 135.255 60.96 0)
+			(effects
+				(font
+					(size 1.27 1.27)
+				)
+			)
+		)
+		(property "Footprint" "easyeda2kicad:LL-34_L3.5-W1.5-RD"
+			(at 134.62 58.42 0)
+			(effects
+				(font
+					(size 1.27 1.27)
+				)
+				(hide yes)
+			)
+		)
+		(property "Datasheet" "https://lcsc.com/product-detail/Zener-Diodes_ZMM33_C8082.html"
+			(at 134.62 55.88 0)
+			(effects
+				(font
+					(size 1.27 1.27)
+				)
+				(hide yes)
+			)
+		)
+		(property "Description" ""
+			(at 134.62 66.04 0)
+			(effects
+				(font
+					(size 1.27 1.27)
+				)
+				(hide yes)
+			)
+		)
+		(property "LCSC Part" "C8082"
+			(at 134.62 53.34 0)
+			(effects
+				(font
+					(size 1.27 1.27)
+				)
+				(hide yes)
+			)
+		)
+		(pin "2"
+		)
+		(pin "1"
+		)
+		(instances
+			(project "GraduateProject"
+				(path "/5608137a-e4aa-4fc5-a1c7-a13152d0b864/de7250b6-5542-41da-b336-1d929c24525c"
+					(reference "D5")
+					(unit 1)
+				)
+			)
+		)
+	)
+	(symbol
 		(lib_id "Device:C")
 		(at 95.25 82.55 270)
@@
 				(path "/5608137a-e4aa-4fc5-a1c7-a13152d0b864/de7250b6-5542-41da-b336-1d929c24525c"
 					(reference "C1")
-					(unit 1)
-				)
-			)
-		)
-	)
-	(symbol
-		(lib_id "Diode:BZV55B36")
-		(at 135.89 66.04 0)
-		(mirror y)
-		(unit 1)
-		(exclude_from_sim no)
-		(in_bom yes)
-		(on_board yes)
-		(dnp no)
-		(property "Reference" "D3"
-			(at 138.684 71.882 0)
-			(effects
-				(font
-					(size 1.27 1.27)
-				)
-				(justify left)
-			)
-		)
-		(property "Value" "BZV55B36"
-			(at 138.684 69.342 0)
-			(effects
-				(font
-					(size 1.27 1.27)
-				)
-				(justify left)
-			)
-		)
-		(property "Footprint" "Diode_SMD:D_MiniMELF"
-			(at 135.89 70.485 0)
-			(effects
-				(font
-					(size 1.27 1.27)
-				)
-				(hide yes)
-			)
-		)
-		(property "Datasheet" "https://assets.nexperia.com/documents/data-sheet/BZV55_SER.pdf"
-			(at 135.89 66.04 0)
-			(effects
-				(font
-					(size 1.27 1.27)
-				)
-				(hide yes)
-			)
-		)
-		(property "Description" "36V, 500mW, 2%, Zener diode, MiniMELF"
-			(at 135.89 66.04 0)
-			(effects
-				(font
-					(size 1.27 1.27)
-				)
-				(hide yes)
-			)
-		)
-		(property "JLCPCB" ""
-			(at 135.89 66.04 0)
-			(effects
-				(font
-					(size 1.27 1.27)
-				)
-				(hide yes)
-			)
-		)
-		(pin "2"
-		)
-		(pin "1"
-		)
-		(instances
-			(project "GraduateProject"
-				(path "/5608137a-e4aa-4fc5-a1c7-a13152d0b864/de7250b6-5542-41da-b336-1d929c24525c"
-					(reference "D3")
 					(unit 1)
 				)
@@
 	(symbol
 		(lib_id "power:GND")
-		(at 125.73 69.85 0)
+		(at 123.19 69.85 0)
 		(unit 1)
 		(exclude_from_sim no)
@@
 		(dnp no)
 		(property "Reference" "#PWR08"
-			(at 125.73 76.2 0)
+			(at 123.19 76.2 0)
 			(effects
 				(font
@@
 		)
 		(property "Value" "GND"
-			(at 125.73 74.168 0)
+			(at 123.19 74.168 0)
 			(effects
 				(font
@@
 		)
 		(property "Footprint" ""
-			(at 125.73 69.85 0)
+			(at 123.19 69.85 0)
 			(effects
 				(font
@@
 		)
 		(property "Datasheet" ""
-			(at 125.73 69.85 0)
+			(at 123.19 69.85 0)
 			(effects
 				(font
@@
 		)
 		(property "Description" "Power symbol creates a global label with name \"GND\" , ground"
-			(at 125.73 69.85 0)
-			(effects
-				(font
+			(at 123.19 69.85 0)
+			(effects
+				(font

Commit message: Add files via upload
17h37 11/9/2025
Parts:
- removed U1: TLP181GB-S, easyeda2kicad:SOP-4_L3.7-W4.6-P2.54-LS7.0-TL, symbol easyeda2kicad:TLP181GB-S
- removed U2, U3: 78L05G-AB3-R, Package_TO_SOT_SMD:SOT-89-3, symbol Regulator_Linear:KA78M05_TO252
- removed U4: 26V-15V L78L15ABUTR, easyeda2kicad:SOT-89-3_L4.5-W2.5-P1.50-LS4.2-TL, symbol easyeda2kicad:L78L15ABUTR
- added U2: L7815, Package_TO_SOT_SMD:TO-263-2, symbol Regulator_Linear:L7815
- added U3, U4: L7805, Package_TO_SOT_SMD:TO-263-2, symbol Regulator_Linear:L7805
- added U6: EL357N(D)(TA)-G_C42385002, easyeda2kicad:SOP-4_L3.9-W4.4-P2.54-LS7.0-TL, symbol easyeda2kicad:EL357N(D)(TA)-G_C42385002
- D5: value ZMM33_C8082 35V -> ZMM36_C8082 35V
Connections:
- net 5V_PIC1: now also U3.3 (OUT)
- net 5V_PIC2: now also U4.3 (OUT)
- net GND: now also U2.2 (GND), U3.2 (GND), U4.2 (GND), U6.3 (EM)
- net RA4_T0CKI: now also U6.4 (COL)
- net at R9.1, TU4.1: now also U2.3 (OUT)
- net at C4.1, C5.1, C7.1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: now also U2.1 (IN), U3.1 (IN), U4.1 (IN)
- net at C2.2, R6.1, R7.2: now also U6.1 (AN)
- net at C2.1, C3.2, J2.4 (Pin_4)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: now also U6.2 (CAT)

Commit message: Add files via upload
18h02 12/9/25
Connections:
- net +26V: now also D5.2 (A), TU3.1; no longer D5.1 (C), TU3.2
- net GND: now also D5.1 (C), TU3.2; no longer D5.2 (A), TU3.1
Other:
- moved on the sheet: D5
Changed lines of the file:
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@@
 	(symbol
 		(lib_id "easyeda2kicad:ZMM33_C8082")
-		(at 134.62 66.04 180)
+		(at 134.62 66.04 0)
+		(mirror x)
 		(unit 1)
 		(exclude_from_sim no)
@@
 		(on_board yes)
 		(dnp no)
-		(fields_autoplaced yes)
 		(property "Reference" "D5"
-			(at 135.255 58.42 0)
+			(at 133.985 58.42 0)
 			(effects
 				(font
@@
 		)
 		(property "Value" "ZMM36_C8082 35V"
-			(at 135.255 60.96 0)
+			(at 133.985 60.96 0)
 			(effects
 				(font
@@
 		(lib_id "easyeda2kicad:TAJB335K035RNJ")
 		(at 160.02 72.39 0)
+		(mirror y)
 		(unit 1)
 		(exclude_from_sim no)
@@
 		(on_board yes)
 		(dnp no)
-		(fields_autoplaced yes)
 		(property "Reference" "TU3"
-			(at 160.655 67.31 0)
+			(at 159.385 67.31 0)
 			(effects
 				(font
@@
 		)
 		(property "Value" "3.3uF 35V"
-			(at 160.655 69.85 0)
-			(effects
-				(font
+			(at 159.385 69.85 0)
+			(effects
+				(font

Commit message: Add files via upload
13/9/25
Changed lines of the file:
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@@
 	(wire
 		(pts
-			(xy 161.29 113.03) (xy 162.56 113.03)
+			(xy 157.48 113.03) (xy 162.56 113.03)
 		)
 		(stroke
@@
 	(symbol
 		(lib_id "power:GND")
-		(at 161.29 113.03 0)
+		(at 157.48 113.03 0)
 		(unit 1)
 		(exclude_from_sim no)
@@
 		(dnp no)
 		(property "Reference" "#PWR014"
-			(at 161.29 119.38 0)
+			(at 157.48 119.38 0)
 			(effects
 				(font
@@
 		)
 		(property "Value" "GND"
-			(at 161.29 117.348 0)
+			(at 157.48 117.348 0)
 			(effects
 				(font
@@
 		)
 		(property "Footprint" ""
-			(at 161.29 113.03 0)
+			(at 157.48 113.03 0)
 			(effects
 				(font
@@
 		)
 		(property "Datasheet" ""
-			(at 161.29 113.03 0)
+			(at 157.48 113.03 0)
 			(effects
 				(font
@@
 		)
 		(property "Description" "Power symbol creates a global label with name \"GND\" , ground"
-			(at 161.29 113.03 0)
+			(at 157.48 113.03 0)
 			(effects
 				(font

Commit message: Add files via upload
5/10/25
Parts:
- removed U2: L7815, Package_TO_SOT_SMD:TO-263-2, symbol Regulator_Linear:L7815
- removed U3, U4: L7805, Package_TO_SOT_SMD:TO-263-2, symbol Regulator_Linear:L7805
- removed U6: EL357N(D)(TA)-G_C42385002, easyeda2kicad:SOP-4_L3.9-W4.4-P2.54-LS7.0-TL, symbol easyeda2kicad:EL357N(D)(TA)-G_C42385002
- added U1, U3: LM7805T, easyeda2kicad:TO-220-3_L10.0-W4.5-P2.54-L, symbol easyeda2kicad:LM7805T
- added U2: TLP181GB-S, easyeda2kicad:SOP-4_L3.7-W4.6-P2.54-LS7.0-TL, symbol easyeda2kicad:TLP181GB-S
- added U4: L7815CV, easyeda2kicad:TO-220-3_L10.0-W4.5-P2.54-L, symbol easyeda2kicad:L7815CV
- C1: Buying link (none) -> https://www.thegioiic.com/tu-gom-0805-10nf-50v
- C2, C4, C5, C7: Buying link (none) -> https://www.thegioiic.com/tu-gom-0805-1-5nf-50v
- C3: value 50V 68nF ceramic -> 50V 68nF; Buying link (none) -> https://www.thegioiic.com/tu-gom-0805-68nf-50v
- C6: value 50V 10nF ceramic -> 50V 10nF; Buying link (none) -> https://www.thegioiic.com/tu-gom-1206-10nf-50v
- D5: Buying link (none) -> https://www.thegioiic.com/zmm36-diode-zener-36v-500mw-sod-80
- R10: Buying link (none) -> https://www.thegioiic.com/dien-tro-100-ohm-0805-1-
- R11, R6: Buying link (none) -> https://www.thegioiic.com/dien-tro-33-kohm-0805-1-
- R7: Buying link (none) -> https://www.thegioiic.com/dien-tro-3-3-kohm-0805-1-
- R8: Buying link (none) -> https://www.thegioiic.com/dien-tro-10-ohm-0805-1-
- R9: Buying link (none) -> https://www.thegioiic.com/dien-tro-1-kohm-0805-1-
- TU1, TU2: Buying link (none) -> https://www.thegioiic.com/tu-tantalum-10uf-16v-2312-tajc106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
Connections:
- net 5V_PIC1: now also U1.3 (OUT)
- net 5V_PIC2: now also U3.3 (OUT)
- net GND: now also U1.2 (GND), U2.4 (EMI), U3.2 (GND), U4.2 (GND)
- net RA4_T0CKI: now also U2.6 (COL)
- net at C2.2, R6.1, R7.2: now also U2.1 (AN)
- net at C2.1, C3.2, J2.4 (Pin_4)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: now also U2.3 (CAT)
- net at R9.1, TU4.1: now also U4.3 (OUT)
- net at C4.1, C5.1, C7.1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: now also U1.1 (VIN), U3.1 (VIN), U4.1 (IN)
Other:
- moved on the sheet: C1, C2, C3, C4, C5, C6, C7, D4, D5, J2, R10, R11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
