File: GraduateProject/Relays.kicad_sch (KiCad schematic)
At the start: 13 parts, among them J1 Conn_01x05_Pin, Q13 MMBTRA101SS, Q14 MMBTRA101SS, Q15 MMBTRA101SS

Commit message: Add files via upload
10/9/25
Parts:
- J1: footprint (none) -> Connector_PinHeader_2.54mm:PinHeader_1x05_P2.54mm_Vertical
- renumbered D6 to D1, D5 to D2, Q15 to Q1, Q14 to Q2, Q13 to Q3, R43 to R1, R40 to R2, R41 to R3, R35 to R4, R34 to R5, REL2 to REL1, REL1 to REL2
Changed lines of the file:
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@@
+	(wire
+		(pts
+			(xy 101.6 93.98) (xy 104.14 93.98)
+		)
+		(stroke
+			(width 0)
+			(type default)
+		)
+	)
 	(wire
 		(pts
@@
 		(on_board yes)
 		(dnp no)
-		(property "Reference" "R40"
+		(property "Reference" "R2"
 			(at 124.968 124.46 90)
 			(effects
@@
 		(property "Description" "Resistor"
 			(at 127 125.73 0)
+			(effects
+				(font
+					(size 1.27 1.27)
+				)
+				(hide yes)
+			)
+		)
+		(property "JLCPCB" ""
+			(at 127 125.73 90)
 			(effects
 				(font
@@
 			(project "GraduateProject"
 				(path "/5608137a-e4aa-4fc5-a1c7-a13152d0b864/b81b2d94-1e34-4e7a-a495-c468ec4a4433"
-					(reference "R40")
+					(reference "R2")
 					(unit 1)
 				)
@@
 		(on_board yes)
 		(dnp no)
-		(property "Reference" "R34"
+		(property "Reference" "R5"
 			(at 174.752 137.16 90)
 			(effects
@@
 		(property "Description" "Resistor"
 			(at 172.72 135.89 0)
+			(effects
+				(font
+					(size 1.27 1.27)
+				)
+				(hide yes)
+			)
+		)
+		(property "JLCPCB" ""
+			(at 172.72 135.89 90)
 			(effects
 				(font
@@
 			(project "GraduateProject"
 				(path "/5608137a-e4aa-4fc5-a1c7-a13152d0b864/b81b2d94-1e34-4e7a-a495-c468ec4a4433"
-					(reference "R34")
+					(reference "R5")
 					(unit 1)
 				)
@@
 		(on_board yes)
 		(dnp no)
-		(property "Reference" "#PWR019"
+		(property "Reference" "#PWR02"
 			(at 107.95 143.51 0)
 			(effects
@@
 			(project "GraduateProject"
 				(path "/5608137a-e4aa-4fc5-a1c7-a13152d0b864/b81b2d94-1e34-4e7a-a495-c468ec4a4433"
-					(reference "#PWR019")
+					(reference "#PWR02")
 					(unit 1)
 				)
@@
 		(on_board yes)
 		(dnp no)
-		(property "Reference" "REL1"
+		(property "Reference" "REL2"
 			(at 142.24 91.44 90)
 			(effects
@@
 		(property "LCSC Part" "C1564084"
 			(at 124.46 100.33 0)
+			(effects
+				(font
+					(size 1.27 1.27)
+				)
+				(hide yes)
+			)
+		)
+		(property "JLCPCB" ""
+			(at 142.24 100.33 90)
 			(effects
 				(font
@@
 			(project "GraduateProject"
 				(path "/5608137a-e4aa-4fc5-a1c7-a13152d0b864/b81b2d94-1e34-4e7a-a495-c468ec4a4433"
-					(reference "REL1")
+					(reference "REL2")
 					(unit 1)
 				)
@@
 		(on_board yes)
 		(dnp no)
-		(property "Reference" "Q13"
+		(property "Reference" "Q3"
 			(at 161.29 127 90)
 			(effects
@@
 		(property "LCSC Part" "C3588808"
 			(at 180.34 139.7 0)
+			(effects
+				(font
+					(size 1.27 1.27)
+				)
+				(hide yes)
+			)
+		)
+		(property "JLCPCB" ""
+			(at 162.56 139.7 90)
 			(effects
 				(font
@@
 			(project "GraduateProject"
 				(path "/5608137a-e4aa-4fc5-a1c7-a13152d0b864/b81b2d94-1e34-4e7a-a495-c468ec4a4433"
-					(reference "Q13")
+					(reference "Q3")
 					(unit 1)
 				)
@@
 		(dnp no)
 		(fields_autoplaced yes)
-		(property "Reference" "Q15"
+		(property "Reference" "Q1"
 			(at 109.22 121.9199 0)
 			(effects
@@
 		(property "LCSC Part" "C3588808"
 			(at 100.33 142.24 0)
+			(effects
+				(font
+					(size 1.27 1.27)
+				)
+				(hide yes)
+			)
+		)
+		(property "JLCPCB" ""
+			(at 100.33 124.46 0)
 			(effects
 				(font
@@
 			(project "GraduateProject"
 				(path "/5608137a-e4aa-4fc5-a1c7-a13152d0b864/b81b2d94-1e34-4e7a-a495-c468ec4a4433"
-					(reference "Q15")
+					(reference "Q1")
 					(unit 1)
 				)
@@
 		(on_board yes)
 		(dnp no)
-		(property "Reference" "R43"
+		(property "Reference" "R1"
 			(at 100.33 135.128 90)
 			(effects
@@
 		(property "Description" "Resistor"
 			(at 99.06 137.16 0)
+			(effects
+				(font
+					(size 1.27 1.27)
+				)
+				(hide yes)
+			)
+		)
+		(property "JLCPCB" ""
+			(at 99.06 137.16 90)
 			(effects
 				(font
@@
 			(project "GraduateProject"
 				(path "/5608137a-e4aa-4fc5-a1c7-a13152d0b864/b81b2d94-1e34-4e7a-a495-c468ec4a4433"
-					(reference "R43")
+					(reference "R1")
 					(unit 1)
 				)
@@
 		(dnp no)
 		(fields_autoplaced yes)
-		(property "Reference" "D5"
+		(property "Reference" "D2"
 			(at 142.24 109.22 0)
 			(effects
@@
 		)
 		(property "Description" "36V, 500mW, 2%, Zener diode, MiniMELF"
+			(at 142.24 114.3 0)
+			(effects
+				(font
+					(size 1.27 1.27)
+				)
+				(hide yes)
+			)
+		)
+		(property "JLCPCB" ""
 			(at 142.24 114.3 0)
 			(effects
@@
 			(project "GraduateProject"
 				(path "/5608137a-e4aa-4fc5-a1c7-a13152d0b864/b81b2d94-1e34-4e7a-a495-c468ec4a4433"
-					(reference "D5")
+					(reference "D2")
 					(unit 1)
 				)
@@
 		(dnp no)
 		(fields_autoplaced yes)
-		(property "Reference" "D6"
+		(property "Reference" "D1"
 			(at 113.03 105.41 0)
 			(effects
@@
 		)
 		(property "Description" "36V, 500mW, 2%, Zener diode, MiniMELF"
+			(at 113.03 110.49 0)
+			(effects
+				(font
+					(size 1.27 1.27)
+				)
+				(hide yes)
+			)
+		)
+		(property "JLCPCB" ""
 			(at 113.03 110.49 0)
 			(effects
@@
 			(project "GraduateProject"
 				(path "/5608137a-e4aa-4fc5-a1c7-a13152d0b864/b81b2d94-1e34-4e7a-a495-c468ec4a4433"
-					(reference "D6")
+					(reference "D1")
 					(unit 1)
 				)
@@
 			)
 		)
-		(property "Footprint" ""
+		(property "Footprint" "Connector_PinHeader_2.54mm:PinHeader_1x05_P2.54mm_Vertical"
 			(at 115.57 48.26 0)
 			(effects
@@
 		(property "Description" "Generic connector, single row, 01x05, script generated"
 			(at 115.57 48.26 0)
+			(effects
+				(font
+					(size 1.27 1.27)
+				)
+				(hide yes)
+			)
+		)
+		(property "JLCPCB" ""
+			(at 115.57 48.26 90)
 			(effects
 				(font
@@
 		(on_board yes)
 		(dnp no)
-		(property "Reference" "REL2"
+		(property "Reference" "REL1"
 			(at 114.046 80.772 90)
 			(effects
@@
 		(property "LCSC Part" "C1564084"
 			(at 96.52 88.9 0)
+			(effects
+				(font
+					(size 1.27 1.27)
+				)
+				(hide yes)
+			)
+		)
+		(property "JLCPCB" ""
+			(at 114.3 88.9 90)
 			(effects
 				(font
@@
 			(project "GraduateProject"
 				(path "/5608137a-e4aa-4fc5-a1c7-a13152d0b864/b81b2d94-1e34-4e7a-a495-c468ec4a4433"
-					(reference "REL2")
+					(reference "REL1")
 					(unit 1)
 				)
@@
 		(on_board yes)
 		(dnp no)
-		(property "Reference" "#PWR033"
+		(property "Reference" "#PWR04"
 			(at 125.73 105.41 0)
 			(effects
@@
 			(project "GraduateProject"
 				(path "/5608137a-e4aa-4fc5-a1c7-a13152d0b864/b81b2d94-1e34-4e7a-a495-c468ec4a4433"
-					(reference "#PWR033")
+					(reference "#PWR04")
 					(unit 1)
 				)
@@
 	(symbol
 		(lib_id "power:GND")
-		(at 104.14 93.98 270)
+		(at 101.6 93.98 270)
 		(unit 1)
 		(exclude_from_sim no)
@@
 		(on_board yes)
 		(dnp no)
-		(property "Reference" "#PWR032"
-			(at 97.79 93.98 0)
+		(property "Reference" "#PWR01"
+			(at 95.25 93.98 0)
 			(effects
 				(font
@@
 		)
 		(property "Value" "GND"
-			(at 99.822 93.98 0)
+			(at 97.282 93.98 0)
 			(effects
 				(font
@@
 		)
 		(property "Footprint" ""
-			(at 104.14 93.98 0)
+			(at 101.6 93.98 0)
 			(effects
 				(font
@@
 		)
 		(property "Datasheet" ""
-			(at 104.14 93.98 0)
+			(at 101.6 93.98 0)
 			(effects
 				(font
@@
 		)
 		(property "Description" "Power symbol creates a global label with name \"GND\" , ground"
-			(at 104.14 93.98 0)
+			(at 101.6 93.98 0)
 			(effects
 				(font
@@
 			(project "GraduateProject"
 				(path "/5608137a-e4aa-4fc5-a1c7-a13152d0b864/b81b2d94-1e34-4e7a-a495-c468ec4a4433"
-					(reference "#PWR032")
+					(reference "#PWR01")
 					(unit 1)
 				)
@@
 		(on_board yes)
 		(dnp no)
-		(property "Reference" "#PWR029"
+		(property "Reference" "#PWR05"
 			(at 177.8 139.7 0)
 			(effects
@@
 			(project "GraduateProject"
 				(path "/5608137a-e4aa-4fc5-a1c7-a13152d0b864/b81b2d94-1e34-4e7a-a495-c468ec4a4433"
-					(reference "#PWR029")
+					(reference "#PWR05")
 					(unit 1)
 				)
@@
 		(on_board yes)
 		(dnp no)
-		(property "Reference" "R41"
+		(property "Reference" "R3"
 			(at 130.048 127 90)
 			(effects
@@
 		(property "Description" "Resistor"
 			(at 132.08 128.27 0)
+			(effects
+				(font
+					(size 1.27 1.27)
+				)
+				(hide yes)
+			)
+		)
+		(property "JLCPCB" ""
+			(at 132.08 128.27 90)
 			(effects
 				(font
@@
 			(project "GraduateProject"
 				(path "/5608137a-e4aa-4fc5-a1c7-a13152d0b864/b81b2d94-1e34-4e7a-a495-c468ec4a4433"
-					(reference "R41")
+					(reference "R3")
 					(unit 1)
 				)
@@
 		(on_board yes)
 		(dnp no)
-		(property "Reference" "R35"
+		(property "Reference" "R4"
 			(at 156.21 146.558 90)
 			(effects
@@
 		(property "Description" "Resistor"
 			(at 154.94 148.59 0)
+			(effects
+				(font
+					(size 1.27 1.27)
+				)
+				(hide yes)
+			)
+		)
+		(property "JLCPCB" ""
+			(at 154.94 148.59 90)
 			(effects
 				(font
@@
 			(project "GraduateProject"
 				(path "/5608137a-e4aa-4fc5-a1c7-a13152d0b864/b81b2d94-1e34-4e7a-a495-c468ec4a4433"
-					(reference "R35")
+					(reference "R4")
 					(unit 1)
 				)
@@
 		(on_board yes)
 		(dnp no)
-		(property "Reference" "#PWR018"
+		(property "Reference" "#PWR03"
 			(at 127 137.16 0)
 			(effects
@@
 			(project "GraduateProject"
 				(path "/5608137a-e4aa-4fc5-a1c7-a13152d0b864/b81b2d94-1e34-4e7a-a495-c468ec4a4433"
-					(reference "#PWR018")
+					(reference "#PWR03")
 					(unit 1)
 				)
@@
 		(dnp no)
 		(fields_autoplaced yes)
-		(property "Reference" "Q14"
+		(property "Reference" "Q2"
 			(at 149.86 121.9199 0)
 			(effects
@@
 		(property "LCSC Part" "C3588808"
 			(at 140.97 142.24 0)
+			(effects
+				(font
+					(size 1.27 1.27)
+				)
+				(hide yes)
+			)
+		)
+		(property "JLCPCB" ""
+			(at 140.97 124.46 0)
 			(effects
 				(font
@@
 			(project "GraduateProject"
 				(path "/5608137a-e4aa-4fc5-a1c7-a13152d0b864/b81b2d94-1e34-4e7a-a495-c468ec4a4433"
-					(reference "Q14")
+					(reference "Q2")
 					(unit 1)
 				)

Commit message: Add files via upload
11/9/25
Parts:
- removed D1, D2: BZV55B36, Diode_SMD:D_MiniMELF, symbol Diode:BZV55B36
- removed Q1, Q2, Q3: MMBTRA101SS, easyeda2kicad:SOT-23-3_L2.9-W1.3-P1.90-LS2.4-BR, symbol easyeda2kicad:MMBTRA101SS
- added D1, D3: ZMM33_C8082 35V, easyeda2kicad:LL-34_L3.5-W1.5-RD, symbol easyeda2kicad:ZMM33_C8082
- added Q1, Q11, Q2: BC846 1BT-NPN, Package_TO_SOT_SMD:SOT-23, symbol Transistor_BJT:BC846
Connections:
- net GND: now also D1.2 (A), D3.2 (A), Q11.2 (E), Q2.2 (E)
- net RB1_PIC1: now also Q11.1 (B)
- net at R2.2, R3.2: now also Q1.1 (B)
- net at R4.2, R5.2: now also Q2.1 (B)
- net at REL2.A1: now also D1.1 (C), Q1.3 (C)
- net at REL1.A1: now also D3.1 (C), Q11.3 (C)
- new net: Q1.2 (E), Q2.3 (C)

Commit message: Add files via upload
17h37 11/9/2025
Parts:
- removed Q1, Q11, Q2: BC846 1BT-NPN, Package_TO_SOT_SMD:SOT-23, symbol Transistor_BJT:BC846
- added Q1, Q11, Q36: MMBT2222A, Package_TO_SOT_SMD:SOT-23, symbol Transistor_BJT:MMBT2222A
- D1, D3: value ZMM33_C8082 35V -> ZMM36_C8082 35V
Connections:
- net GND: now also Q1.2 (E), Q36.2 (E)
- net RB1_PIC1: now also Q36.1 (B)
- net at R2.2, R3.2: now also Q11.1 (B)
- net at R4.2, R5.2: now also Q1.1 (B)
- net at D1.1 (C), REL2.A1: now also Q11.3 (C)
- net at D3.1 (C), REL1.A1: now also Q36.3 (C)
- new net: Q1.3 (C), Q11.2 (E)

Commit message: Add files via upload
5/10/25
Parts:
- removed Q1, Q11, Q36: MMBT2222A, Package_TO_SOT_SMD:SOT-23, symbol Transistor_BJT:MMBT2222A
- added Q11, Q36, Q4: BCX56, Package_TO_SOT_SMD:SOT-89-3, symbol Transistor_BJT:BCX56
- D1, D3: Buying link (none) -> https://www.thegioiic.com/zmm36-diode-zener-36v-500mw-sod-80
- R1, R3, R4: Buying link (none) -> https://www.thegioiic.com/dien-tro-1-kohm-0805-1-
- R2, R5: Buying link (none) -> https://www.thegioiic.com/dien-tro-4-7-kohm-0805-1-
Connections:
- net GND: now also Q36.3 (E), Q4.3 (E)
- net RB1_PIC1: now also Q4.1 (B)
- net at R2.2, R3.2: now also Q11.1 (B)
- net at R4.2, R5.2: now also Q36.1 (B)
- net at D1.1 (C), REL2.A1: now also Q11.2 (C)
- net at D3.1 (C), REL1.A1: now also Q4.2 (C)
- new net: Q11.3 (E), Q36.2 (C)
