File: GraduateProject/GraduateProject-backups/GraduateProject-2025-09-11_214900/GraduateProject.kicad_pcb (KiCad board)
At the start: 2 copper layers, 90 x 70 mm, 143 parts, among them IC1 PIC16C620A-04/SS, IC2 PIC16C620A-04/SS, J1 Conn_01x05_Pin, J2 Conn_01x04_Pin, J5 Conn_01x04_Pin, J6 Conn_01x04_Pin, J7 Conn_01x05_Pin, J8 Conn_01x05_Pin, Q1 MMBT2222A, Q10 IMX1T110, Q11 MMBT2222A, Q12 IMX1T110, Q13 IMX1T110, Q14 IMX1T110, Q15 IMX1T110, Q16 MMBT2222A, Q17 MMBT2222A, Q18 MMBT2222A, Q19 MMBT2222A, Q2 MMBT2222A, Q20 MMBT2222A, Q21 MMBT2222A, Q22 MMBT2222A, Q23 MMBT3906, Q24 MMBT2222A, Q25 MMBT2222A, Q26 MMBT3906, Q27 MMBT2222A, Q28 MMBT2222A, Q29 MMBT2222A, Q3 MBT3946DW1T1, Q30 MMBT2222A, Q31 MMBT2222A, Q32 MMBT2222A, Q33 MMBT2222A, Q34 MMBT2222A, Q35 MMBT2222A, Q36 MMBT2222A, Q4 MMBT2222A, Q6 IMX1T110, Q7 IMX1T110, Q8 MBT3946DW1T1, Q9 IMX1T110, SW1 SS12D10G3, U2 L7815, U3 L7805, U4 L7805, U5 B0505S-1W, U6 EL357N(D)(TA)-G_C42385002, U7 B0505S-1W

Commit message: Add files via upload
18h02 12/9/25
Parts:
- moved Q17 35.3 mm to (178.9, 103.8), turned to 0 degrees
- moved R51 34.2 mm to (178.6, 106.4), turned to 180 degrees
- moved Q21 31.5 mm to (146.6, 115.7)
- moved Q10 31.5 mm to (146.6, 111.9)
- moved Q22 31.5 mm to (146.6, 108.2)
- moved R45 31.3 mm to (182.2, 105.8), turned to 90 degrees
- moved R43 30.7 mm to (184.2, 105.8), turned to 90 degrees
- moved R44 30.6 mm to (186.2, 105.8), turned to 90 degrees
- moved C23 27.5 mm to (164.1, 116.1), turned to 0 degrees
- moved R52 27.3 mm to (175.2, 108.3), turned to 180 degrees
- moved Q12 27.3 mm to (175.1, 105.4), turned to 90 degrees
- moved C17 26.4 mm to (170.6, 122.0), turned to 180 degrees
- moved R46 25.1 mm to (186.8, 108.6), turned to 0 degrees
- moved C19 24.9 mm to (171.7, 99.8), turned to 180 degrees
- moved C21 24.6 mm to (155.5, 113.9)
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Connections:
- D5 pad 1: GND -> +26V
- D5 pad 2: +26V -> GND
- TU3 pad 1: +26V -> GND
- TU3 pad 2: GND -> +26V
Routing:
- net Net-(U2-IN): track 115.0 -> 0.00 mm, vias 6 -> 0
- net /PICs/5V_PIC1: track 112.4 -> 0.00 mm, vias 2 -> 0
- net /CONNECTORS/CONN_J3_4: track 92.6 -> 0.00 mm, vias 6 -> 0
- net +26V: track 91.1 -> 0.00 mm, vias 2 -> 0
- net /CONNECTORS/RB3_PIC1: track 73.0 -> 0.00 mm, vias 6 -> 0
- net /CONNECTORS/Q10_B1: track 72.2 -> 0.00 mm, vias 10 -> 0
- net /CONNECTORS/Q10_B2: track 71.8 -> 0.00 mm, vias 6 -> 0
- net /PICs/5V_PIC2: track 71.6 -> 0.00 mm, vias 6 -> 0
- net Net-(J7-Pin_2): track 68.6 -> 0.00 mm, vias 2 -> 0
- net /CONNECTORS/RB4_PIC1: track 66.9 -> 0.00 mm, vias 6 -> 0
- net GND: track 62.4 -> 0.00 mm, vias 63 -> 0
- net /CONNECTORS/CONN_J2_4: track 60.4 -> 0.00 mm, vias 2 -> 0
- net /CONNECTORS/Q12_E2: track 59.8 -> 0.00 mm, vias 9 -> 0
- net /PICs/RA4_T0CKI: track 59.6 -> 0.00 mm, vias 2 -> 0
- net /CONNECTORS/Q14_C2: track 56.5 -> 0.00 mm, vias 6 -> 0
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- removed copper zone on B.Cu, net GND
- removed copper zone on F.Cu, net GND
Other:
- outline, holes or cut-outs redrawn
- board text added: "48.5mm"
- board text removed: "14.6mm"
- board text removed: "35mm"
