File: GraduateProject/GraduateProject-backups/GraduateProject-2025-09-11_214900/GraduateProject.kicad_sch (KiCad schematic)
At the start: 0 parts

Commit message: Add files via upload
18h02 12/9/25
Changed lines of the file:
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@@
 	(wire
 		(pts
-			(xy 168.91 58.42) (xy 195.58 58.42)
-		)
-		(stroke
-			(width 0)
-			(type default)
-		)
-	)
-	(wire
-		(pts
-			(xy 168.91 66.04) (xy 198.12 66.04)
+			(xy 167.64 58.42) (xy 195.58 58.42)
+		)
+		(stroke
+			(width 0)
+			(type default)
+		)
+	)
+	(wire
+		(pts
+			(xy 167.64 66.04) (xy 198.12 66.04)
 		)
 		(stroke
@@
 	(wire
 		(pts
-			(xy 133.35 68.58) (xy 128.27 68.58)
+			(xy 132.08 68.58) (xy 128.27 68.58)
 		)
 		(stroke
@@
 	(wire
 		(pts
-			(xy 168.91 73.66) (xy 200.66 73.66)
-		)
-		(stroke
-			(width 0)
-			(type default)
-		)
-	)
-	(wire
-		(pts
-			(xy 168.91 55.88) (xy 204.47 55.88)
+			(xy 167.64 73.66) (xy 200.66 73.66)
+		)
+		(stroke
+			(width 0)
+			(type default)
+		)
+	)
+	(wire
+		(pts
+			(xy 167.64 55.88) (xy 204.47 55.88)
 		)
 		(stroke
@@
 	(wire
 		(pts
-			(xy 99.06 55.88) (xy 133.35 55.88)
+			(xy 99.06 55.88) (xy 132.08 55.88)
 		)
 		(stroke
@@
 	(wire
 		(pts
-			(xy 168.91 68.58) (xy 199.39 68.58)
+			(xy 167.64 68.58) (xy 199.39 68.58)
 		)
 		(stroke
@@
 	(wire
 		(pts
-			(xy 118.11 52.07) (xy 133.35 52.07)
+			(xy 118.11 52.07) (xy 132.08 52.07)
 		)
 		(stroke
@@
 	(wire
 		(pts
-			(xy 133.35 73.66) (xy 130.81 73.66)
-		)
-		(stroke
-			(width 0)
-			(type default)
-		)
-	)
-	(wire
-		(pts
-			(xy 78.74 43.18) (xy 133.35 43.18)
+			(xy 132.08 73.66) (xy 130.81 73.66)
+		)
+		(stroke
+			(width 0)
+			(type default)
+		)
+	)
+	(wire
+		(pts
+			(xy 78.74 43.18) (xy 132.08 43.18)
 		)
 		(stroke
@@
 	(wire
 		(pts
-			(xy 133.35 63.5) (xy 125.73 63.5)
-		)
-		(stroke
-			(width 0)
-			(type default)
-		)
-	)
-	(wire
-		(pts
-			(xy 133.35 48.26) (xy 124.46 48.26)
+			(xy 132.08 63.5) (xy 125.73 63.5)
+		)
+		(stroke
+			(width 0)
+			(type default)
+		)
+	)
+	(wire
+		(pts
+			(xy 132.08 48.26) (xy 124.46 48.26)
 		)
 		(stroke
@@
 	(wire
 		(pts
-			(xy 133.35 71.12) (xy 129.54 71.12)
+			(xy 132.08 71.12) (xy 129.54 71.12)
 		)
 		(stroke
@@
 	(wire
 		(pts
-			(xy 133.35 60.96) (xy 102.87 60.96)
+			(xy 132.08 60.96) (xy 102.87 60.96)
 		)
 		(stroke
@@
 	(wire
 		(pts
-			(xy 133.35 58.42) (xy 119.38 58.42)
+			(xy 132.08 58.42) (xy 119.38 58.42)
 		)
 		(stroke
@@
 	(wire
 		(pts
-			(xy 168.91 60.96) (xy 196.85 60.96)
+			(xy 167.64 60.96) (xy 196.85 60.96)
 		)
 		(stroke
@@
 	(wire
 		(pts
-			(xy 78.74 45.72) (xy 133.35 45.72)
-		)
-		(stroke
-			(width 0)
-			(type default)
-		)
-	)
-	(wire
-		(pts
-			(xy 133.35 66.04) (xy 127 66.04)
+			(xy 78.74 45.72) (xy 132.08 45.72)
+		)
+		(stroke
+			(width 0)
+			(type default)
+		)
+	)
+	(wire
+		(pts
+			(xy 132.08 66.04) (xy 127 66.04)
 		)
 		(stroke
@@
 	)
 	(sheet
-		(at 133.35 40.132)
+		(at 132.08 40.132)
 		(size 35.56 37.592)
 		(exclude_from_sim no)
@@
 		)
 		(property "Sheetname" "PICs"
-			(at 133.35 39.4204 0)
+			(at 132.08 39.4204 0)
 			(effects
 				(font
@@
 		)
 		(property "Sheetfile" "PICs.kicad_sch"
-			(at 133.35 78.3086 0)
+			(at 132.08 78.3086 0)
 			(effects
 				(font
@@
 		)
 		(pin "5V_PIC1" input
-			(at 133.35 43.18 180)
+			(at 132.08 43.18 180)
 			(effects
 				(font
@@
 		)
 		(pin "5V_PIC2" input
-			(at 133.35 45.72 180)
+			(at 132.08 45.72 180)
 			(effects
 				(font
@@
 		)
 		(pin "CONN_J3_4" input
-			(at 133.35 48.26 180)
+			(at 132.08 48.26 180)
 			(effects
 				(font
@@
 		)
 		(pin "RA2_PIC1" output
-			(at 133.35 58.42 180)
+			(at 132.08 58.42 180)
 			(effects
 				(font
@@
 		)
 		(pin "RA2_PIC2" input
-			(at 168.91 58.42 0)
+			(at 167.64 58.42 0)
 			(effects
 				(font
@@
 		)
 		(pin "RA4_T0CKI" input
-			(at 133.35 52.07 180)
+			(at 132.08 52.07 180)
 			(effects
 				(font
@@
 		)
 		(pin "RB1_PIC1" input
-			(at 133.35 55.88 180)
+			(at 132.08 55.88 180)
 			(effects
 				(font
@@
 		)
 		(pin "RB1_PIC2" input
-			(at 168.91 55.88 0)
+			(at 167.64 55.88 0)
 			(effects
 				(font
@@
 		)
 		(pin "RB2_PIC1" input
-			(at 133.35 60.96 180)
+			(at 132.08 60.96 180)
 			(effects
 				(font
@@
 		)
 		(pin "RB3_PIC1" input
-			(at 133.35 63.5 180)
+			(at 132.08 63.5 180)
 			(effects
 				(font
@@
 		)
 		(pin "RB3_PIC2" input
-			(at 168.91 60.96 0)
+			(at 167.64 60.96 0)
 			(effects
 				(font
@@
 		)
 		(pin "RB4_PIC1" input
-			(at 133.35 66.04 180)
+			(at 132.08 66.04 180)
 			(effects
 				(font
@@
 		)
 		(pin "RB4_PIC2" input
-			(at 168.91 66.04 0)
+			(at 167.64 66.04 0)
 			(effects
 				(font
@@
 		)
 		(pin "RB5_PIC1" input
-			(at 133.35 68.58 180)
+			(at 132.08 68.58 180)
 			(effects
 				(font
@@
 		)
 		(pin "RB6_PIC1" input
-			(at 133.35 71.12 180)
+			(at 132.08 71.12 180)
 			(effects
 				(font
@@
 		)
 		(pin "RB6_PIC2" input
-			(at 168.91 68.58 0)
+			(at 167.64 68.58 0)
 			(effects
 				(font
@@
 		)
 		(pin "RB7_PIC1" input
-			(at 133.35 73.66 180)
+			(at 132.08 73.66 180)
 			(effects
 				(font
@@
 		)
 		(pin "RB7_PIC2" input
-			(at 168.91 73.66 0)
-			(effects
-				(font
+			(at 167.64 73.66 0)
+			(effects
+				(font
