File: GraduateProject/GraduateProject-backups/GraduateProject-2025-09-11_214900/PICs.kicad_sch (KiCad schematic)
At the start: 24 parts, among them IC1 PIC16C620A-04/SS, IC2 PIC16C620A-04/SS, Q4 MMBT2222A, SW1 SS12D10G3, U5 B0505S-1W, U7 B0505S-1W

Commit message: Add files via upload
18h02 12/9/25
Changed lines of the file:
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@@
-	(wire
-		(pts
-			(xy 128.27 43.18) (xy 132.08 43.18)
-		)
-		(stroke
-			(width 0)
-			(type default)
-		)
-	)
 	(wire
 		(pts
@@
 	(hierarchical_label "5V_PIC2"
 		(shape input)
-		(at 128.27 43.18 180)
-		(effects
-			(font
+		(at 132.08 43.18 180)
+		(effects
+			(font
