File: Connector/Connector.kicad_pcb (KiCad board)
At the start: 2 copper layers, 25 x 13 mm, 5 parts, among them J2 Conn_01x05_Pin, J3 Conn_01x01_Pin, J4 Conn_01x01_Pin, J5 Conn_01x01_Pin, J6 Conn_01x01_Pin

Commit message: Add files via upload
13/9/25
Routing:
- net Net-(J2-Pin_2): track 6.55 -> 7.23 mm
Other:
- board size 25 x 13 mm -> 25 x 13.5 mm
Changed lines of the file:
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@@
 			)
 		)
-		(pad "1" thru_hole rect
+		(pad "1" connect rect
 			(at 0 0)
-			(size 1.7 1.7)
-			(drill 1)
-			(layers "*.Cu" "*.Mask")
-			(remove_unused_layers no)
+			(size 1.7 4)
+			(layers "F.Cu" "F.Mask")
 			(net 1 "Net-(J2-Pin_2)")
 			(pinfunction "Pin_1")
@@
 			)
 		)
-		(pad "1" thru_hole rect
+		(pad "1" connect rect
 			(at 0 0)
-			(size 1.7 1.7)
-			(drill 1)
-			(layers "*.Cu" "*.Mask")
-			(remove_unused_layers no)
+			(size 1.7 4)
+			(layers "F.Cu" "F.Mask")
 			(net 4 "Net-(J2-Pin_4)")
 			(pinfunction "Pin_1")
@@
 			)
 		)
-		(pad "1" thru_hole rect
+		(pad "1" connect rect
 			(at 0 0)
-			(size 1.7 1.7)
-			(drill 1)
-			(layers "*.Cu" "*.Mask")
-			(remove_unused_layers no)
+			(size 1.7 4)
+			(layers "F.Cu" "F.Mask")
 			(net 3 "Net-(J2-Pin_5)")
 			(pinfunction "Pin_1")
@@
 			)
 		)
-		(pad "1" thru_hole rect
+		(pad "1" connect rect
 			(at 0 0)
-			(size 1.7 1.7)
-			(drill 1)
-			(layers "*.Cu" "*.Mask")
-			(remove_unused_layers no)
+			(size 6 2.5)
+			(layers "F.Cu" "F.Mask")
 			(net 5 "unconnected-(J2-Pin_1-Pad1)")
 			(pinfunction "Pin_1")
 			(pintype "passive+no_connect")
 		)
-		(pad "2" thru_hole circle
+		(pad "2" connect rect
 			(at 0 2.54)
-			(size 1.7 1.7)
-			(drill 1)
-			(layers "*.Cu" "*.Mask")
-			(remove_unused_layers no)
+			(size 6 1.7)
+			(layers "F.Cu" "F.Mask")
 			(net 1 "Net-(J2-Pin_2)")
 			(pinfunction "Pin_2")
 			(pintype "passive")
 		)
-		(pad "3" thru_hole circle
+		(pad "3" connect rect
 			(at 0 5.08)
-			(size 1.7 1.7)
-			(drill 1)
-			(layers "*.Cu" "*.Mask")
-			(remove_unused_layers no)
+			(size 6 1.7)
+			(layers "F.Cu" "F.Mask")
 			(net 2 "Net-(J2-Pin_3)")
 			(pinfunction "Pin_3")
 			(pintype "passive")
 		)
-		(pad "4" thru_hole circle
+		(pad "4" connect rect
 			(at 0 7.62)
-			(size 1.7 1.7)
-			(drill 1)
-			(layers "*.Cu" "*.Mask")
-			(remove_unused_layers no)
+			(size 6 1.7)
+			(layers "F.Cu" "F.Mask")
 			(net 4 "Net-(J2-Pin_4)")
 			(pinfunction "Pin_4")
 			(pintype "passive")
 		)
-		(pad "5" thru_hole circle
+		(pad "e" connect rect
 			(at 0 10.16)
-			(size 1.7 1.7)
-			(drill 1)
-			(layers "*.Cu" "*.Mask")
-			(remove_unused_layers no)
+			(size 6 1.7)
+			(layers "F.Cu" "F.Mask")
 			(net 3 "Net-(J2-Pin_5)")
 			(pinfunction "Pin_5")
@@
 			)
 		)
-		(pad "1" thru_hole rect
+		(pad "1" connect rect
 			(at 0 0)
-			(size 1.7 1.7)
-			(drill 1)
-			(layers "*.Cu" "*.Mask")
-			(remove_unused_layers no)
+			(size 1.7 4)
+			(layers "F.Cu" "F.Mask")
 			(net 2 "Net-(J2-Pin_3)")
 			(pinfunction "Pin_1")
@@
 	(gr_rect
 		(start 90 105)
-		(end 115 118)
+		(end 115 118.5)
 		(stroke
 			(width 0.05)
@@
 	)
 	(segment
-		(start 94.46 109.04)
-		(end 97 106.5)
+		(start 97 106.5)
+		(end 97 107.652)
 		(width 2)
 		(layer "F.Cu")
@@
 	)
 	(segment
-		(start 91.5 109.04)
-		(end 94.46 109.04)
+		(start 95.612 109.04)
+		(end 91.5 109.04)
+		(width 2)
+		(layer "F.Cu")
+		(net 1)
+	)
+	(segment
+		(start 97 107.652)
+		(end 95.612 109.04)
 		(width 2)
 		(layer "F.Cu")
@@
 	)
 	(segment
+		(start 91.5 116.66)
+		(end 103.34 116.66)
+		(width 2)
+		(layer "F.Cu")
+		(net 3)
+	)
+	(segment
 		(start 103.34 116.66)
 		(end 113.5 106.5)
@@
 	)
 	(segment
-		(start 91.5 116.66)
-		(end 103.34 116.66)
+		(start 91.5 114.12)
+		(end 100.38 114.12)
 		(width 2)
 		(layer "F.Cu")
-		(net 3)
+		(net 4)
 	)
 	(segment
@@
 		(width 2)
 		(layer "F.Cu")
-		(net 4)
-	)
-	(segment
-		(start 91.5 114.12)
-		(end 100.38 114.12)
-		(width 2)
-		(layer "F.Cu")
